Commit message: add robot controller and test commands

File: my_arm_robot_description/urdf/arm_robot_gazebo.urdf.xacro (robot description, xacro)
@@ -6,5 +6,5 @@
         <robot_param>robot_description</robot_param>
         <robot_param>robot_state_publisher</robot_param>
-        <parameters></parameters>
+        <parameters>$(find my_arm_robot_controller)/config/arm_robot_conrollers.yaml</parameters>
     </plugin>
 </gazebo>

File: my_arm_robot_description/urdf/arm_robot_ros2_control.urdf.xacro (robot description, xacro)
@@ -8,6 +8,6 @@
     <joint name ="joint_1">
     <command_interface name = "position">
-        <params name="min">-${PI/2}</params>
-        <params name = "max">${PI/2}</params>
+        <param name="min">-${PI/2}</param>
+        <param name = "max">${PI/2}</param>
     </command_interface>
     <state_interface name ="position" />
@@ -15,6 +15,6 @@
         <joint name ="joint_2">
     <command_interface name = "position">
-        <params name="min">-${PI/2}</params>
-        <params name = "max">${PI/2}</params>
+        <param name="min">-${PI/2}</param>
+        <param name = "max">${PI/2}</param>
     </command_interface>
     <state_interface name ="position" />
@@ -22,6 +22,6 @@
         <joint name ="joint_3">
     <command_interface name = "position">
-        <params name="min">-${PI/2}</params>
-        <params name = "max">${PI/2}</params>
+        <param name="min">-${PI/2}</param>
+        <param name = "max">${PI/2}</param>
     </command_interface>
     <state_interface name ="position" />
@@ -29,15 +29,15 @@
         <joint name ="joint_4">
     <command_interface name = "position">
-        <params name="min">-${PI/2}</params>
-        <params name = "max">0.0</params>
+        <param name="min">-${PI/2}</param>
+        <param name = "max">0.0</param>
     </command_interface>
     <state_interface name ="position" />
     </joint>
         <joint name ="joint_5">
-        <params name = "mimic">joint_4</params>
-        <params name = "multiplier">-1</params>
+        <param name = "mimic">joint_4</param>
+        <param name = "multiplier">-1</param>
         <command_interface name = "position">
-            <params name="min">0.0</params>
-            <params name = "max">${PI/2}</params>
+            <param name="min">0.0</param>
+            <param name = "max">${PI/2}</param>
         </command_interface>
     <state_interface name ="position" />

File: my_arm_robot_description/urdf/model.urdf.xacro (robot description, xacro)
@@ -177,5 +177,5 @@
         <origin xyz="-0.08 0.13 -0.1"/>
             <mimic joint="joint_4" multiplier="-1"/>
-        <limit lower="0.0" upper="${PI/2}" effort="${effort}" velocity="${velocity/2}"/>
+        <limit lower="0.0" upper="${PI / 2}" effort="${effort}" velocity="${velocity}"/>
     </joint>
 <xacro:default_transimssion number = "1"/>
