Commit message: digital twin for yaskawa MHLF

File: yaskawa_mh5_description/motoman_resources/models/common_materials.xacro (robot description, xacro)
@@ -1,5 +1,5 @@
 <?xml version="1.0" ?>
 <robot xmlns:xacro="http://ros.org/wiki/xacro">
-  <xacro:include filename="$(find motoman_resources)/urdf/common_colors.xacro"/>
+  <xacro:include filename="$(find yaskawa_mh5_description)/motoman_resources/models/common_colors.xacro"/>
   <xacro:macro name="material_yaskawa_blue">
     <material name="">

File: yaskawa_mh5_description/urdf/mh5.urdf.xacro (robot description, xacro)
@@ -4,7 +4,33 @@
 <!-- |    EDITING THIS FILE BY HAND IS NOT RECOMMENDED                                 | -->
 <!-- =================================================================================== -->
-<robot name="yaskawa_mh5" xmlns:xacro="http://ros.org/wiki/xacro">
+<robot name="yaskawa_mh5lf" xmlns:xacro="http://ros.org/wiki/xacro">
+  <xacro:include filename="$(find yaskawa_mh5_description)/urdf/mh5_gazebo.urdf.xacro"/>
+  <xacro:include filename="$(find yaskawa_mh5_description)/urdf/mh5_ros2_controller.urdf.xacro"/>
+<!-- macro function for inertial-->
+	<xacro:macro name="default_inertial" params="mass">
+		<inertial>
+			<mass value="${mass}"/>
+			<inertia ixx="1.0" ixy="0.0" ixz="0.0"
+					iyy="1.0" iyz="0.0"
+					izz="1.0" />
+		</inertial>
+	</xacro:macro>
+<!-- end of macro function for inertial -->
+<!-- transmission for robot controller -->
+  <xacro:macro name="default_transmission" params="number">
+      <transmission name="transmission_${number}">
+          <plugin>transmission_interface/SimpleTransmission</plugin>
+          <actuator name="motor_${number}" role="actuator1">
+              <joint name="joint_${number}" role="joint1">
+                  <mechanical_reduction>1.0</mechanical_reduction>
+              </joint>
+          </actuator>
+      </transmission>
+  </xacro:macro>
+<!-- end transmission for robot controller -->
   <!-- link list -->
+  <link name = "world" />
   <link name="base_link">
+    <xacro:default_inertial mass="1.0"/>
     <visual>
       <origin rpy="0 0 3.14159"/>
@@ -27,4 +53,5 @@
   </link>
   <link name="link_s">
+    <xacro:default_inertial mass="1.0"/>
     <visual>
       <geometry>
@@ -43,4 +70,5 @@
   </link>
   <link name="link_l">
+    <xacro:default_inertial mass="1.0"/>
     <visual>
       <!-- <origin rpy="1.57 3.1416 0" xyz="0 0 0"/> -->
@@ -56,7 +84,8 @@
       </geometry>
       <material name="yellow"/>
-    </collision>
+      robot</collision>
   </link>
   <link name="link_u">
+    <xacro:default_inertial mass="1.0"/>
     <visual>
       <!-- <origin rpy="1.57 -3.1415 0" xyz="0 0 0"/> -->
@@ -75,4 +104,5 @@
   </link>
   <link name="link_r">
+    <xacro:default_inertial mass="1.0"/>
     <visual>
       <!-- <origin rpy="0 0 3.1416" xyz="0 0 0"/> -->
@@ -91,4 +121,5 @@
   </link>
   <link name="link_b">
+    <xacro:default_inertial mass="1.0"/>
     <visual>
       <!-- <origin rpy="-1.57 0 3.1416" xyz="0 0 0"/> -->
@@ -107,4 +138,5 @@
   </link>
   <link name="link_t">
+    <xacro:default_inertial mass="1.0"/>
     <visual>
       <geometry>
@@ -122,4 +154,11 @@
   <!-- end of link list -->
   <!-- joint list -->
+  <joint name="virtual_joint" type="fixed">
+    <origin xyz="0.0 0.0 0.0" rpy="0.0 0.0 0.0"/>
+    <parent link="world"/>
+    <child link="base_link"/>
+    <axis xyz="0.0 0.0 0.0"/>
+    <limit lower="0.0" upper="0.0" effort="0.0" velocity="0.0"/>
+  </joint>
   <joint name="joint_s" type="revolute">
     <parent link="base_link"/>
@@ -158,5 +197,5 @@
   </joint>
   <joint name="joint_t" type="revolute">
-    <parent link="link_b"/>
+    <parent link="link_b"/>"
     <child link="link_t"/>
     <origin rpy="0 0 0" xyz="0.0865 0 0"/>
@@ -164,3 +203,10 @@
     <limit effort="100" lower="-6.2831" upper="6.2831" velocity="6.97"/>
   </joint>
+  <!-- Define transmissions -->
+    <xacro:default_transmission number="s"/>
+    <xacro:default_transmission number="l"/>
+    <xacro:default_transmission number="u"/>
+    <xacro:default_transmission number="r"/>
+    <xacro:default_transmission number="b"/>
+    <xacro:default_transmission number="t"/>
 </robot>

File: yaskawa_mh5_description/urdf/mh5_gazebo.urdf.xacro (robot description, xacro)
@@ -1,9 +1,8 @@
 <?xml version="1.0"?>
-<robot xmlns:xacro="http://ros.org/wiki/xacro" name="yaskawa_mh5">
+<robot xmlns:xacro="http://ros.org/wiki/xacro" name="yaskawa_mh5lf">
     <gazebo>
         <plugin filename="libgazebo_ros2_control.so" name="gazebo_ros2_control">
             <robot_param>robot_description</robot_param>
-            <robot_param>robot_state_publisher</robot_param>
-            <!-- <parameters></parameters>  -->
+            <robot_param_node>robot_state_publisher</robot_param_node>
             <parameters>$(find yaskawa_mh5_controller)/config/mh5_ros2_controller.yaml</parameters>
         </plugin>

File: yaskawa_mh5_description/urdf/unused_mh5.urdf.xacro (robot description, xacro)
@@ -1,5 +1,5 @@
 <?xml version="1.0" ?>
 <robot name="yaskawa_mh5lf" xmlns:xacro="http://ros.org/wiki/xacro">
-	<xacro:include filename="$(find yaskawa_mh5_description)/urdf/mh5_macro.xacro" />
+	<xacro:include filename="$(find yaskawa_mh5_description)/urdf/mh5_macro.urdf.xacro" />
 	<xacro:yaskawa_mh5_description prefix=""/>
 </robot>
