Commit message: new updates

File: yaskawa_mh5_description/urdf/mh5.urdf.xacro (robot description, xacro)
@@ -52,4 +52,48 @@
     </collision>
   </link>
+<!-- Camera Pole Link -->
+<!-- <link name="camera_pole">
+  <xacro:default_inertial mass="0.5"/>
+  <visual>
+    <origin xyz="1 0 0"/>
+    <geometry>
+      <cylinder length="1.0" radius="0.05"/>
+    </geometry>
+    <material name="grey">
+      <color rgba="0.5 0.5 0.5 1.0"/>
+    </material>
+  </visual>
+  <collision>
+    <origin xyz="1 0 0"/>
+    <geometry>
+      <cylinder length="1.0" radius="0.05"/>
+    </geometry>
+  </collision>
+</link> -->
+<!-- Depth Camera Link -->
+<!--
+<link name="depth_camera">
+  <xacro:default_inertial mass="0.5"/>
+  <visual>
+    <geometry>
+      <box size="0.2 0.4 0.1"/>
+    </geometry>
+    <material name="black">
+      <color rgba="0.0 0.0 0.0 1.0"/>
+    </material>
+  </visual>
+  <collision>
+    <geometry>
+      <box size="0.2 0.4 0.1"/>
+    </geometry>
+  </collision>
+</link> -->
+<!-- Joint between camera pole and depth camera -->
+<!-- <joint name="pole_to_camera" type="fixed">
+  <parent link="camera_pole"/>
+  <child link="depth_camera"/>
+  <origin xyz="0 0 0.95" rpy="0 0 0"/>
+  <axis xyz="0 1.5 0"/>
+</joint>  -->
   <link name="link_s">
     <xacro:default_inertial mass="1.0"/>
@@ -96,5 +140,4 @@
     </visual>
     <collision>
-      <!-- <origin rpy="1.57 -3.1415 0" xyz="0 0 0"/> -->
       <geometry>
         <mesh filename="package://yaskawa_mh5_description/meshes/mh5/collision/MH5_U_AXIS.stl"/>
@@ -106,5 +149,4 @@
     <xacro:default_inertial mass="1.0"/>
     <visual>
-      <!-- <origin rpy="0 0 3.1416" xyz="0 0 0"/> -->
       <geometry>
         <mesh filename="package://yaskawa_mh5_description/meshes/mh5/visual/MH5_R_AXIS.stl"/>
@@ -113,5 +155,4 @@
     </visual>
     <collision>
-      <!-- <origin rpy="0 0 3.1416" xyz="0 0 0"/> -->
       <geometry>
         <mesh filename="package://yaskawa_mh5_description/meshes/mh5/collision/MH5_R_AXIS.stl"/>
@@ -120,8 +161,23 @@
     </collision>
   </link>
+<!-- 3D sensor  -->
+  <link name="3d_camera">
+    <xacro:default_inertial mass="0.5"/>
+    <visual>
+      <geometry>
+          <mesh filename = "package://yaskawa_mh5_description/meshes/mh5/collision/BIN_PICKING_MODULE_1CH_ASM.stl" scale="0.001 0.001 0.001"/>
+      </geometry>
+      <material name="silver"/>
+    </visual>
+    <collision>
+      <geometry>
+        <mesh filename = "package://yaskawa_mh5_description/meshes/mh5/collision/BIN_PICKING_MODULE_1CH_ASM.stl" scale="0.001 0.001 0.001"/>
+      </geometry>
+      <material name="silver"/>
+    </collision>
+  </link>
   <link name="link_b">
     <xacro:default_inertial mass="1.0"/>
     <visual>
-      <!-- <origin rpy="-1.57 0 3.1416" xyz="0 0 0"/> -->
       <geometry>
         <mesh filename="package://yaskawa_mh5_description/meshes/mh5/visual/MH5_B_AXIS.stl"/>
@@ -130,5 +186,4 @@
     </visual>
     <collision>
-      <!-- <origin rpy="-1.57 0 3.1416" xyz="0 0 0"/> -->
       <geometry>
         <mesh filename="package://yaskawa_mh5_description/meshes/mh5/collision/MH5_B_AXIS.stl"/>
@@ -152,6 +207,4 @@
     </collision>
   </link>
-  <!-- end of link list -->
-  <!-- joint list -->
   <joint name="virtual_joint" type="fixed">
     <origin xyz="0.0 0.0 0.0" rpy="0.0 0.0 0.0"/>
@@ -160,4 +213,10 @@
     <axis xyz="0.0 0.0 0.0"/>
     <limit lower="0.0" upper="0.0" effort="0.0" velocity="0.0"/>
+  </joint>
+  <!-- Joint between link_r and camera  -->
+  <joint name="joint_3d_camera" type="fixed">
+    <parent link="link_r"/>
+    <child link="3d_camera"/>
+    <origin xyz="0.0715 0 0.08" rpy="1.5708 0 1.5708"/>
   </joint>
   <joint name="joint_s" type="revolute">

File: yaskawa_mh5_description/urdf/mh5_gazebo.urdf.xacro (robot description, xacro)
@@ -7,4 +7,25 @@
             <parameters>$(find yaskawa_mh5_controller)/config/mh5_ros2_controller.yaml</parameters>
         </plugin>
+        <plugin name="gazebo_ros_depth_camera" filename="libgazebo_ros_depth_camera.so">
+            <always_on>true</always_on>
+            <update_rate>30.0</update_rate>
+            <camera_name>depth_camera</camera_name>
+            <image_topic_name>/depth_camera/image_raw</image_topic_name>
+            <camera_info_topic_name>/depth_camera/camera_info</camera_info_topic_name>
+            <frame_name>depth_camera</frame_name>
+            <hack_baseline>0.07</hack_baseline>
+            <distortion_k1>0.0</distortion_k1>
+            <distortion_k2>0.0</distortion_k2>
+            <distortion_k3>0.0</distortion_k3>
+            <distortion_t1>0.0</distortion_t1>
+            <distortion_t2>0.0</distortion_t2>
+            <horizontal_fov>1.047</horizontal_fov>
+            <image_width>640</image_width>
+            <image_height>480</image_height>
+            <clip>
+              <near>0.1</near>
+              <far>10.0</far>
+            </clip>
+          </plugin>
     </gazebo>
 </robot>
