Commit message: gripper condigiration has been added for testing purpose

File: src/yaskawa_mh5_description/urdf/TesseraVue_3D_sensor_bigger.urdf.xacro (robot description, xacro)
@@ -15,5 +15,5 @@
     <parent link="link_r"/>
     <child link="tesseravue_chassis_link"/>
-    <origin xyz="0.2 0.0 0.01" rpy="1.5708 0 1.5708"/> <!-- Adjust as needed -->
+    <origin xyz="0.0715 0.05 0.08" rpy="1.5708 0 1.5708"/> <!-- Adjust as needed -->
   </joint>
   <!-- 3D sensor -->
@@ -21,12 +21,12 @@
     <xacro:default_inertial mass="0.5"/>
     <visual>
-    <origin xyz="0.02 0.07 0.01" rpy="0 0 0"/>
+    <origin xyz="0 0.05 0.3" rpy="0 0 0"/>
       <geometry>
-        <mesh filename="package://yaskawa_mh5_description/meshes/mh5/collision/BIN_PICKING_MODULE_1CH_ASM.stl" scale="0.001 0.001 0.001"/>
+        <mesh filename="package://yaskawa_mh5_description/meshes/mh5/collision/BIN_PICKING_MODULE_1CH_ASM.stl" scale="0.0015 0.0015 0.0015"/>
       </geometry>
     </visual>
     <collision>
       <geometry>
-        <mesh filename="package://yaskawa_mh5_description/meshes/mh5/collision/BIN_PICKING_MODULE_1CH_ASM.stl" scale="0.001 0.001 0.001"/>
+        <mesh filename="package://yaskawa_mh5_description/meshes/mh5/collision/BIN_PICKING_MODULE_1CH_ASM.stl" scale="0.0015 0.0015 0.0015"/>
       </geometry>
     </collision>
@@ -37,7 +37,8 @@
     <parent link="tesseravue_chassis_link"/>
     <child link="tesseravue_camera_link"/>
-    <origin xyz="0.0765 0 0.06" rpy="0 -1.5708 0"/>
+    <origin xyz="0.096 0.07 0.38" rpy="0 -1.5708 0"/>
+    <!-- <origin xyz="0.0765 0 0.06" rpy="0 0 0"/> Adjust as needed -->
   </joint>
- <link name="tesseravue_camera_link">
+  <link name="tesseravue_camera_link">
     <xacro:default_inertial mass="0.5"/>
     <visual>
@@ -53,5 +54,6 @@
     <child link="3dcamera_optical"/>
     <origin xyz="0 0 0" rpy="0 0 0"/>
-    <origin xyz="0 0 0" rpy="-1.5708 0 -1.5708"/>
+    <!-- <origin xyz="0 0 0" rpy="-1.5708 0 -1.5708"/>  -->
+    <origin xyz="0 0 0" rpy="${-PI/2} 0 ${-PI/2}"/>
   </joint>
   <link name="3dcamera_optical"/>

File: src/yaskawa_mh5_description/urdf/grippers.urdf.xacro (robot description, xacro)
@@ -1,48 +1,270 @@
 <?xml version="1.0" ?>
-<robot xmlns:xacro="http://ros.org/wiki/xacro">
-    <xacro:property name="PI" value="3.14159"/>
-    <xacro:property name="effort" value="30.0"/>
-    <xacro:property name="velocity" value="10.0"/>
-    <!-- Macro function for inertial -->
-    <xacro:macro name="default_inertial" params="mass">
-        <inertial>
-            <mass value="${mass}"/>
-            <inertia ixx="1.0" ixy="0.0" ixz="0.0"
-                     iyy="1.0" iyz="0.0"
-                     izz="1.0" />
-        </inertial>
-    </xacro:macro>
-    <!-- Fingers Visualization on Gazebo  -->
-    <link name="gripper_right">
-        <visual>
-            <origin rpy="0 0 0" xyz="0.03 0 0"/>
-            <geometry>
-                <mesh filename="package://yaskawa_mh5_description/meshes/mh5/collision/finger_right.stl" scale="0.002 0.005 0.005" />
-            </geometry>
-        </visual>
-    </link>
-    <link name="gripper_left">
-        <visual>
-            <origin rpy="0 0 0" xyz="0.03 0 0"/>
-            <geometry>
-                <mesh filename="package://yaskawa_mh5_description/meshes/mh5/collision/finger_left.stl" scale="0.002 0.005 0.005" />
-            </geometry>
-        </visual>
-    </link>
-    <!-- Gripper joints -->
-    <joint name="joint_a" type="revolute">
+<robot  xmlns:xacro="http://ros.org/wiki/xacro">
+    <!-- <xacro:property name="PI" value="3.141592654" /> -->
+    <xacro:include filename="$(find rg2_description)/urdf/rg2.gazebo.xacro" />
+    <xacro:include filename="$(find rg2_description)/urdf/rg2.transmissions.xacro" />
+    <!-- <link name="base_link">
+    </link> -->
+    <joint name="base_fixed_joint" type="fixed">
         <parent link="link_t"/>
-        <child link="gripper_right"/>
-        <axis xyz="0 0 1"/>
-        <origin rpy="0 0 0" xyz="0 0 0"/>
-        <limit lower="-${PI/2}" upper="0.0" effort="${effort}" velocity="${velocity}"/>
-    </joint>
-    <joint name="joint_y" type="revolute">
-        <parent link="link_t"/>
-        <child link="gripper_left"/>
-        <axis xyz="0 0 1"/>
-        <origin rpy="0 0 0" xyz="0 0 0"/>
-        <limit lower="0.0" upper="${PI/2}" effort="${effort}" velocity="${velocity}"/>
-        <mimic joint="joint_a" multiplier="-1"/>
-    </joint>
+        <child link="hand_link"/>
+        <origin xyz="0.000 0.000 0.000" rpy="0 0 0"/>
+    </joint>
+    <link name="hand_link">
+        <collision>
+            <origin xyz="0.00 0.00 0.00" rpy="0.00 0.00 0.00"/>
+            <geometry>
+                <mesh filename="package://yaskawa_mh5_description/meshes/rg_gripper/collision/RG2_Hand_col.STL"/>
+            </geometry>
+        </collision>
+        <visual>
+            <origin xyz="0.00 0.00 0.00" rpy="0.00 0.00 0.00"/>
+            <geometry>
+                <mesh filename="package://yaskawa_mh5_description/meshes/rg_gripper/visual/RG2_Hand_vis.STL"/>
+            </geometry>
+        </visual>
+        <!-- <inertial>
+            <origin xyz="0.058091 0.000192 -0.000016" rpy="0.00 0.00 0.00"/>
+            <mass value="0.524520"/>
+            <inertia ixx="0.000193" ixy="0.000000" ixz="0.000000"
+                     iyy="0.000564" iyz="-0.000001"hand_link
+                     izz="0.000636" />
+        </inertial> -->
+        <inertial>
+            <origin xyz="0.061902 0.000129 -0.000005" rpy="0.00 0.00 0.00"/>
+            <mass value="1.684558"/>
+            <inertia ixx="0.000862" ixy="0.000000" ixz="0.000000"
+                     iyy="0.002401" iyz="-0.000001"
+                     izz="0.002620" />
+        </inertial>
+    </link>
+    <!-- Jari Kiri -->
+    <joint name="gripper_joint" type="revolute">
+        <parent link="hand_link"/>
+        <child link="l_moment_arm_link"/>
+        <origin xyz="0.105 0.017 0.010" rpy="0 0 0"/>
+        <axis xyz="0 0 1"/>
+        <limit velocity="3.14" effort="10.6" lower="${-0.45}" upper="${pi*0.5}" />
+        <!-- <limit velocity="3.14" effort="100" lower="-3" upper="3" /> -->
+        <dynamics damping="0.1" friction="0.0" />
+        <implicitSpringDamper>True</implicitSpringDamper>
+    </joint>
+    <xacro:insert_transmission name="gripper_joint" />
+    <link name="l_moment_arm_link">
+        <collision>
+            <origin xyz="0.00 0.00 0.00" rpy="0.00 0.00 0.00"/>
+            <geometry>
+                <mesh filename="package://yaskawa_mh5_description/meshes/rg_gripper/collision/RG2_LeftMomentArm_col.STL"/>
+            </geometry>
+        </collision>
+        <visual>
+            <origin xyz="0.00 0.00 0.00" rpy="0.00 0.00 0.00"/>
+            <geometry>
+                <mesh filename="package://yaskawa_mh5_description/meshes/rg_gripper/visual/RG2_LeftMomentArm_vis.STL"/>
+            </geometry>
+        </visual>
+        <inertial>
+            <origin xyz="0.017004 0.006397 -0.010300" rpy="0.00 0.00 0.00"/>
+            <mass value="0.160209"/>
+            <inertia ixx="0.000023" ixy="0.000019" ixz="0.000000"
+                     iyy="0.000072" iyz="0.000000"
+                     izz="0.000083" />
+        </inertial>
+    </link>
+    <joint name="l_finger_2_joint" type="revolute">
+        <parent link="l_moment_arm_link"/>hand_link
+        <child link="l_finger_link"/>
+        <origin xyz="0.049 0.026 0.000" rpy="0 0 0"/>
+        <axis xyz="0 0 1"/>
+        <limit velocity="3.14" effort="10.6" lower="${-pi*0.5}" upper="${pi*0.5}" />
+        <!-- <limit velocity="3.14" effort="100" lower="-3" upper="3" /> -->
+        <mimic joint="gripper_joint" multiplier="-1"/>
+        <dynamics damping="0.1" friction="0.0" />
+        <implicitSpringDamper>True</implicitSpringDamper>
+    </joint>
+    <!-- <xacro:insert_transmission name="l_finger_2_joint" /> -->
+    <xacro:mimic_joint_plugin_gazebo name_prefix="l_finger_2_joint"
+                                     parent_joint="gripper_joint"
+                                     mimic_joint="l_finger_2_joint"
+                                     has_pid="false"
+                                     multiplier="-1.0"
+                                     max_effort="10.6" />
+    <link name="l_finger_link">
+        <collision>
+            <origin xyz="0.00 0.00 0.00" rpy="0.00 0.00 0.00"/>
+            <geometry>
+                <mesh filename="package://yaskawa_mh5_description/meshes/rg_gripper/collision/RG2_LeftFinger_col.STL"/>
+            </geometry>
+        </collision>
+        <visual>
+            <origin xyz="0.00 0.00 0.00" rpy="0.00 0.00 0.00"/>
+            <geometry>
+                <mesh filename="package://yaskawa_mh5_description/meshes/rg_gripper/visual/RG2_LeftFinger_vis.STL"/>
+            </geometry>
+        </visual>
+        <inertial>
+            <origin xyz="0.024695 -0.010178 -0.010001" rpy="0.00 0.00 0.00"/>
+            <mass value="0.081638"/>
+            <inertia ixx="0.000006" ixy="-0.000005" ixz="0.000000"
+                     iyy="0.000025" iyz="0.000000"
+                     izz="0.000026" />
+        </inertial>
+    </link>
+    <joint name="l_finger_passive_joint" type="revolute">
+        <parent link="hand_link"/>
+        <child link="l_truss_arm_link"/>
+        <origin xyz="0.122 0.008 0.010" rpy="0 0 0"/>
+        <axis xyz="0 0 1"/>
+        <limit velocity="3.14" effort="10.6" lower="${-pi*0.5}" upper="${pi*0.5}" />
+        <!-- <limit velocity="3.14" effort="100" lower="-3" upper="3" /> -->
+        <mimic joint="gripper_joint" multiplier="1"/>
+        <dynamics damping="0.1" friction="0.0" />
+        <implicitSpringDamper>True</implicitSpringDamper>
+    </joint>
+    <!-- <xacro:insert_transmission name="l_finger_passive_joint" /> -->
+    <xacro:mimic_joint_plugin_gazebo name_prefix="l_finger_passive_joint"
+                                     parent_joint="gripper_joint"
+                                     mimic_joint="l_finger_passive_joint"
+                                     has_pid="false"
+                                     multiplier="1.0"
+                                     max_effort="10.6" />
+    <link name="l_truss_arm_link">
+        <collision>
+            <origin xyz="0.00 0.00 0.00" rpy="0.00 0.00 0.00"/>
+            <geometry>
+                <mesh filename="package://yaskawa_mh5_description/meshes/rg_gripper/collision/RG2_LeftTrussArm_col.STL"/>
+            </geometry>
+        </collision>
+        <visual>
+            <origin xyz="0.00 0.00 0.00" rpy="0.00 0.00 0.00"/>
+            <geometry>
+                <mesh filename="package://yaskawa_mh5_description/meshes/rg_gripper/visual/RG2_LeftTrussArm_vis.STL"/>
+            </geometry>
+        </visual>
+        <inertial>
+            <origin xyz="0.023075 0.012136 -0.010000" rpy="0.00 0.00 0.00"/>
+            <mass value="0.065927"/>
+            <inertia ixx="0.000010" ixy="0.000010" ixz="0.000000"
+                     iyy="0.000024" iyz="0.000000"
+                     izz="0.000025" />
+        </inertial>
+    </link>
+    <!-- Jari Kanan -->
+    <joint name="r_finger_1_joint" type="revolute">
+        <parent link="hand_link"/>
+        <child link="r_moment_arm_link"/>
+        <origin xyz="0.105 -0.017 0.010" rpy="0 0 0"/>
+        <axis xyz="0 0 1"/>
+        <limit velocity="3.14" effort="10.6" lower="${-pi*0.5}" upper="${pi*0.5}" />
+        <!-- <limit velocity="3.14" effort="100" lower="-3" upper="3" /> -->
+        <mimic joint="gripper_joint" multiplier="-1"/>
+        <dynamics damping="0.1" friction="0.0" />
+        <implicitSpringDamper>True</implicitSpringDamper>
+    </joint>
+    <!-- <xacro:insert_transmission name="r_finger_1_joint" /> -->
+    <xacro:mimic_joint_plugin_gazebo name_prefix="r_finger_1_joint"
+                                     parent_joint="gripper_joint"
+                                     mimic_joint="r_finger_1_joint"
+                                     has_pid="false"
+                                     multiplier="-1.0"
+                                     max_effort="10.6" />
+    <link name="r_moment_arm_link">
+        <collision>
+            <origin xyz="0.00 0.00 0.00" rpy="0.00 0.00 0.00"/>
+            <geometry>
+                <mesh filename="package://yaskawa_mh5_description/meshes/rg_gripper/collision/RG2_RightMomentArm_col.STL"/>
+            </geometry>
+        </collision>
+        <visual>
+            <origin xyz="0.00 0.00 0.00" rpy="0.00 0.00 0.00"/>
+            <geometry>
+                <mesh filename="package://yaskawa_mh5_description/meshes/rg_gripper/visual/RG2_RightMomentArm_vis.STL"/>
+            </geometry>
+        </visual>
+        <inertial>
+            <origin xyz="0.017004 -0.006397 -0.010300" rpy="0.00 0.00 0.00"/>
+            <mass value="0.160209"/>
+            <inertia ixx="0.000023" ixy="-0.000019" ixz="0.000000"
+                     iyy="0.000072" iyz="0.000000"
+                     izz="0.000083" />
+        </inertial>
+    </link>
+    <joint name="r_finger_2_joint" type="revolute">
+        <parent link="r_moment_arm_link"/>
+        <child link="r_finger_link"/>
+        <origin xyz="0.049 -0.026 0.000" rpy="0 0 0"/>
+        <axis xyz="0 0 1"/>
+        <limit velocity="3.14" effort="10.6" lower="${-pi*0.5}" upper="${pi*0.5}" />
+        <!-- <limit velocity="3.14" effort="100" lower="-3" upper="3" /> -->
+        <mimic joint="gripper_joint" multiplier="1"/>
+        <dynamics damping="0.1" friction="0.0" />
+        <implicitSpringDamper>True</implicitSpringDamper>
+    </joint>
+    <!-- <xacro:insert_transmission name="r_finger_2_joint" /> -->
+    <xacro:mimic_joint_plugin_gazebo name_prefix="r_finger_2_joint"
+                                     parent_joint="gripper_joint"
+                                     mimic_joint="r_finger_2_joint"
+                                     has_pid="false"
+                                     multiplier="1.0"
+                                     max_effort="10.6" />
+    <link name="r_finger_link">
+        <collision>
+            <origin xyz="0.00 0.00 0.00" rpy="0.00 0.00 0.00"/>
+            <geometry>
+                <mesh filename="package://yaskawa_mh5_description/meshes/rg_gripper/collision/RG2_RightFinger_col.STL"/>
+            </geometry>
+        </collision>
+        <visual>
+            <origin xyz="0.00 0.00 0.00" rpy="0.00 0.00 0.00"/>
+            <geometry>
+                <mesh filename="package://yaskawa_mh5_description/meshes/rg_gripper/visual/RG2_RightFinger_vis.STL"/>
+            </geometry>
+        </visual>
+        <inertial>
+            <origin xyz="0.024695 0.010178 -0.010000" rpy="0.00 0.00 0.00"/>
+            <mass value="0.081637"/>
+            <inertia ixx="0.000006" ixy="0.000005" ixz="0.000000"
+                     iyy="0.000025" iyz="0.000000"
+                     izz="0.000026" />
+        </inertial>
+    </link>
+    <joint name="r_finger_passive_joint" type="revolute">
+        <parent link="hand_link"/>
+        <child link="r_truss_arm_link"/>
+        <origin xyz="0.122 -0.008 0.010" rpy="0 0 0"/>
+        <axis xyz="0 0 1"/>
+        <limit velocity="3.14" effort="10.6" lower="${-pi*0.5}" upper="${pi*0.5}" />
+        <!-- <limit velocity="3.14" effort="100" lower="-3" upper="3" /> -->
+        <mimic joint="gripper_joint" multiplier="-1"/>
+        <dynamics damping="0.1" friction="0.0" />
+        <implicitSpringDamper>True</implicitSpringDamper>
+    </joint>
+    <!-- <xacro:insert_transmission name="r_finger_passive_joint" /> -->
+    <xacro:mimic_joint_plugin_gazebo name_prefix="r_finger_passive_joint"
+                                     parent_joint="gripper_joint"
+                                     mimic_joint="r_finger_passive_joint"
+                                     has_pid="false"
+                                     multiplier="-1.0"
+                                     max_effort="10.6" />
+    <link name="r_truss_arm_link">
+        <collision>
+            <origin xyz="0.00 0.00 0.00" rpy="0.00 0.00 0.00"/>
+            <geometry>
+                <mesh filename="package://yaskawa_mh5_description/meshes/rg_gripper/collision/RG2_RightTrussArm_col.STL"/>
+            </geometry>
+        </collision>
+        <visual>
+            <origin xyz="0.00 0.00 0.00" rpy="0.00 0.00 0.00"/>
+            <geometry>
+                <mesh filename="package://yaskawa_mh5_description/meshes/rg_gripper/visual/RG2_RightTrussArm_vis.STL"/>
+            </geometry>
+        </visual>
+        <inertial>
+            <origin xyz="0.023075 -0.012136 -0.010000" rpy="0.00 0.00 0.00"/>
+            <mass value="0.065927"/>
+            <inertia ixx="0.000010" ixy="-0.000010" ixz="0.000000"
+                     iyy="0.000024" iyz="0.000000"
+                     izz="0.000025" />
+        </inertial>
+    </link>
 </robot>
