Commit message: gripper condigiration has been added for testing purpose

File: src/yaskawa_mh5_description/urdf/mh5.urdf.xacro (robot description, xacro)
@@ -7,6 +7,6 @@
   <xacro:include filename="$(find yaskawa_mh5_description)/urdf/mh5_gazebo.urdf.xacro"/>
   <xacro:include filename="$(find yaskawa_mh5_description)/urdf/mh5_ros2_controller.urdf.xacro"/>
-  <xacro:include filename="$(find yaskawa_mh5_description)/urdf/TesseraVue_3D_sensor.urdf.xacro"/>
-  <xacro:include filename="$(find yaskawa_mh5_description)/urdf/grippers.urdf.xacro"/>
+  <xacro:include filename="$(find yaskawa_mh5_description)/urdf/TesseraVue_3D_sensor_bigger.urdf.xacro"/>
+  <!-- <xacro:include filename="$(find yaskawa_mh5_description)/urdf/grippers.urdf.xacro"/> -->
 <!-- macro function for inertial-->
   <xacro:property name="effort" value="30.0"/>
@@ -41,5 +41,5 @@
      <origin rpy="0 0 0"/>
       <geometry>
-        <mesh filename="package://yaskawa_mh5_description/meshes/mh5/visual/MH5_BASE_AXIS.stl"/>
+        <mesh filename="package://yaskawa_mh5_description/meshes/mh5/visual/MH5_BASE_AXIS.stl" scale="2.0 2.0 2.0"/>
       </geometry>
       <material name="blue">
@@ -50,5 +50,5 @@
       <origin rpy="0 0 3.14159"/>
       <geometry>
-        <mesh filename="package://yaskawa_mh5_description/meshes/mh5/collision/MH5_BASE_AXIS.stl"/>
+        <mesh filename="package://yaskawa_mh5_description/meshes/mh5/collision/MH5_BASE_AXIS.stl" scale="2.0 2.0 2.0"/>
       </geometry>
       <material name="yellow">
@@ -61,5 +61,5 @@
     <visual>
       <geometry>
-        <mesh filename="package://yaskawa_mh5_description/meshes/mh5/visual/MH5_S_AXIS.stl"/>
+        <mesh filename="package://yaskawa_mh5_description/meshes/mh5/visual/MH5_S_AXIS.stl" scale="2.0 2.0 2.0"/>
       </geometry>
       <material name="silver">
@@ -69,5 +69,5 @@
     <collision>
       <geometry>
-        <mesh filename="package://yaskawa_mh5_description/meshes/mh5/collision/MH5_S_AXIS.stl"/>
+        <mesh filename="package://yaskawa_mh5_description/meshes/mh5/collision/MH5_S_AXIS.stl" scale="2.0 2.0 2.0"/>
       </geometry>
       <material name="yellow"/>
@@ -78,5 +78,5 @@
     <visual>
       <geometry>
-        <mesh filename="package://yaskawa_mh5_description/meshes/mh5/visual/MH5_L_AXIS.stl"/>
+        <mesh filename="package://yaskawa_mh5_description/meshes/mh5/visual/MH5_L_AXIS.stl" scale="2.0 2.0 2.0"/>
       </geometry>
       <material name="blue"/>
@@ -84,8 +84,8 @@
     <collision>
       <geometry>
-        <mesh filename="package://yaskawa_mh5_description/meshes/mh5/collision/MH5_L_AXIS.stl"/>
+        <mesh filename="package://yaskawa_mh5_description/meshes/mh5/collision/MH5_L_AXIS.stl" scale="2.0 2.0 2.0"/>
       </geometry>
       <material name="yellow"/>
-      </collision>
+    </collision>
   </link>
   <link name="link_u">
@@ -93,5 +93,5 @@
     <visual>
       <geometry>
-        <mesh filename="package://yaskawa_mh5_description/meshes/mh5/visual/MH5_U_AXIS.stl"/>
+        <mesh filename="package://yaskawa_mh5_description/meshes/mh5/visual/MH5_U_AXIS.stl" scale="2.0 2.0 2.0"/>
       </geometry>
       <material name="blue"/>
@@ -99,5 +99,5 @@
     <collision>
       <geometry>
-        <mesh filename="package://yaskawa_mh5_description/meshes/mh5/collision/MH5_U_AXIS.stl"/>
+        <mesh filename="package://yaskawa_mh5_description/meshes/mh5/collision/MH5_U_AXIS.stl" scale="2.0 2.0 2.0"/>
       </geometry>
       <material name="yellow"/>
@@ -108,5 +108,5 @@
     <visual>
       <geometry>
-        <mesh filename="package://yaskawa_mh5_description/meshes/mh5/visual/MH5_R_AXIS.stl"/>
+        <mesh filename="package://yaskawa_mh5_description/meshes/mh5/visual/MH5_R_AXIS.stl" scale="2.0 2.0 2.0"/>
       </geometry>
       <material name="silver"/>
@@ -114,20 +114,5 @@
     <collision>
       <geometry>
-        <mesh filename="package://yaskawa_mh5_description/meshes/mh5/collision/MH5_R_AXIS.stl"/>
-      </geometry>
-      <material name="yellow"/>
-    </collision>
-  </link>
-  <link name="link_b">
-    <xacro:default_inertial mass="1.0"/>
-    <visual>
-      <geometry>
-        <mesh filename="package://yaskawa_mh5_description/meshes/mh5/visual/MH5_B_AXIS.stl"/>
-      </geometry>
-      <material name="blue"/>
-    </visual>
-    <collision>
-      <geometry>
-        <mesh filename="package://yaskawa_mh5_description/meshes/mh5/collision/MH5_B_AXIS.stl"/>
+        <mesh filename="package://yaskawa_mh5_description/meshes/mh5/collision/MH5_B_AXIS.stl" scale="2.0 2.0 2.0"/>
       </geometry>
       <material name="yellow"/>
@@ -138,5 +123,5 @@
     <visual>
       <geometry>
-        <mesh filename="package://yaskawa_mh5_description/meshes/mh5/visual/MH5_T_AXIS.stl"/>
+        <mesh filename="package://yaskawa_mh5_description/meshes/mh5/visual/MH5_T_AXIS.stl" scale="2.0 2.0 2.0"/>
       </geometry>
       <material name="silver"/>
@@ -144,27 +129,9 @@
     <collision>
       <geometry>
-        <mesh filename="package://yaskawa_mh5_description/meshes/mh5/collision/MH5_T_AXIS.stl"/>
+        <mesh filename="package://yaskawa_mh5_description/meshes/mh5/collision/MH5_T_AXIS.stl" scale="2.0 2.0 2.0"/>
       </geometry>
       <material name="yellow"/>
     </collision>
   </link>
-<!-- Fingers Visualization on Gazebo  -->
-    <!-- <link name="gripper_right">
-        <visual>
-            <origin xyz="00.04 0.5 -0.1" rpy = "0 0 -${PI/2}" />
-            <geometry>
-                <mesh filename="package://yaskawa_mh5_description/meshes/mh5/collision/finger_right.stl" scale="0.002 0.005 0.005" />
-            </geometry>
-        </visual>
-    </link>
-    <link name="gripper_left">
-        <visual>
-        <origin xyz="00.04 0.5 -0.1" rpy = "0 0 -${PI/2}"/>
-            <geometry>
-                <mesh filename="package://yaskawa_mh5_description/meshes/mh5/collision/finger_left.stl" scale="0.002 0.005 0.005" />
-            </geometry>
-        </visual>
-    </link> -->
-<!-- END Fingers Visualization on Gazebo  -->
   <joint name="virtual_joint" type="fixed">
     <origin xyz="0.0 0.0 0.0" rpy="0.0 0.0 0.0"/>
@@ -177,16 +144,12 @@
     <parent link="base_link"/>
     <child link="link_s"/>
-    <origin rpy="0 0 0" xyz="0 0 0.1990"/>
+    <origin rpy="0 0 0" xyz="0 0 0.3980"/>
     <axis xyz="0 0 1"/>
+    <limit effort="100" lower="-1.1345" upper="2.6180" velocity="2.96"/>
+  </joint>
+  <joint name="joint_l" type="revolute">
     <parent link="link_s"/>
     <child link="link_l"/>
-    <origin rpy="0 0 0" xyz="0.0880 0 0.1310"/>
-    <axis xyz="0 1 0"/>
-    <limit effort="100" lower="-1.1345" upper="2.6180" velocity="2.96"/>
-  </joint>
-    <joint name="joint_l" type="revolute">
-    <parent link="link_s"/>
-    <child link="link_l"/>
-    <origin rpy="0 0 0" xyz="0.0880 0 0.1310"/>
+    <origin rpy="0 0 0" xyz="0.1760 0 0.2620"/>
     <axis xyz="0 1 0"/>
     <limit effort="100" lower="-1.1345" upper="2.6180" velocity="2.96"/>
@@ -195,5 +158,5 @@
     <parent link="link_l"/>
     <child link="link_u"/>
-    <origin rpy="0 0 0" xyz="0 0 0.3100"/>
+    <origin rpy="0 0 0" xyz="0 0 0.6200"/>
     <axis xyz="0 -1 0"/>
     <limit effort="100" lower="-1.0122" upper="3.2218" velocity="2.96"/>
@@ -202,5 +165,5 @@
     <parent link="link_u"/>
     <child link="link_r"/>
-    <origin rpy="0 0 0" xyz="0.0715 0 0.0399"/>
+    <origin rpy="0 0 0" xyz="0.1430 0 0.0798"/>
     <axis xyz="-1 0 0"/>
     <limit effort="100" lower="-3.3161" upper="3.3161" velocity="3.48"/>
@@ -209,32 +172,15 @@
     <parent link="link_r"/>
     <child link="link_b"/>
-    <origin rpy="0 0 0" xyz="0.2335 0 0"/>
+    <origin rpy="0 0 0" xyz="0.4670 0 0"/>
     <axis xyz="0 -1 0"/>
     <limit effort="100" lower="-2.1817" upper="2.1817" velocity="3.48"/>
   </joint>
-  <joint name="joint_t" type="revolute">
-    <parent link="link_b"/>"
+  <joint name="joint_t" type="fixed">
+    <parent link="link_b"/>
     <child link="link_t"/>
-    <origin rpy="0 0 0" xyz="0.0865 0 0"/>
-    <axis xyz="-1 0 0"/>
+    <origin rpy="0 0 0" xyz="0.1730 0 0"/>
+    <axis xyz="0 -1 0"/>
     <limit effort="100" lower="-6.2831" upper="6.2831" velocity="6.97"/>
   </joint>
-    <!-- Gripper joints -->
-    <!-- <joint name="joint_a" type="revolute">
-        <parent link="link_t"/>
-        <child link="gripper_right"/>
-        <axis xyz="0 0 1"/>
-        <origin rpy="0 0 0" xyz="0 0 0"/>
-        <limit lower="-1.5708" upper="0.0" effort="100" velocity="3.48"/>
-    </joint>
-    <joint name="joint_y" type="revolute">
-        <parent link="link_t"/>
-        <child link="gripper_left"/>
-        <axis xyz="0 0 1"/>
-        <origin rpy="0 0 0" xyz="0 0 0"/>
-        <limit lower="0.0" upper="1.5708" effort="100" velocity="3.48"/>
-        <mimic joint="joint_a" multiplier="-1"/>
-    </joint> -->
-        <!-- END OF Gripper joints -->
   <!-- Define transmissions -->
     <xacro:default_transmission number="s"/>
@@ -244,5 +190,4 @@
     <xacro:default_transmission number="b"/>
     <xacro:default_transmission number="t"/>
-    <!-- <xacro:default_transmission number="a"/>
-    <xacro:default_transmission number="y"/>     -->
+    <!-- <xacro:default_transmission number="a"/>  -->
 </robot>

File: src/yaskawa_mh5_description/urdf/mh5_ros2_controller.urdf.xacro (robot description, xacro)
@@ -2,4 +2,5 @@
 <robot xmlns:xacro="http://ros.org/wiki/xacro" name="yaskawa_mh5lf">
     <xacro:property name="PI" value="3.14159"/>
+    <!-- <xacro:include filename="$(find yaskawa_mh5_description)/urdf/robotiq_85_gripper.transmission.xacro"/> -->
     <ros2_control name="RobotSystem" type="system">
         <hardware>
@@ -8,12 +9,12 @@
         <joint name="joint_s">
             <command_interface name="position">
-                <param name="min">${-PI/2}</param>
+                <param name="min">-${PI/2}</param>
                 <param name="max">${PI/2}</param>
             </command_interface>
             <state_interface name="position"/>
         </joint>
-        <joint name="joint_l">
+        <joint name="joint_l"><xacro:property name="PI" value="3.14159"/>
             <command_interface name="position">
-                <param name="min">${-PI/2}</param>
+                <param name="min">-${PI/2}</param>
                 <param name="max">${PI/2}</param>
             </command_interface>
@@ -22,5 +23,5 @@
         <joint name="joint_u">
             <command_interface name="position">
-                <param name="min">${-PI/2}</param>
+                <param name="min">-${PI/2}</param><xacro:property name="PI" value="3.14159"/>
                 <param name="max">${PI/2}</param>
             </command_interface>
@@ -29,5 +30,5 @@
         <joint name="joint_r">
             <command_interface name="position">
-                <param name="min">${-PI/2}</param>
+                <param name="min">-${PI/2}</param>
                 <param name="max">${PI/2}</param>
             </command_interface>
@@ -36,5 +37,5 @@
         <joint name="joint_b">
             <command_interface name="position">
-                <param name="min">${-PI/2}</param>
+                <param name="min">-${PI/2}</param>
                 <param name="max">${PI/2}</param>
             </command_interface>
@@ -43,12 +44,4 @@
         <joint name="joint_t">
             <command_interface name="position">
-                <param name="min">${-PI/2}</param>
-                <param name="max">${PI/2}</param>
-            </command_interface>
-            <state_interface name="position"/>
-        </joint>
-    <!-- Gripper -->
-          <joint name="joint_a">
-            <command_interface name="position">
                 <param name="min">-${PI/2}</param>
                 <param name="max">${PI/2}</param>
@@ -56,14 +49,4 @@
             <state_interface name="position"/>
         </joint>
-          <joint name="joint_y">
-          <param name = "mimic">joint_a</param>
-          <param name = "multiplier">-1</param>
-            <command_interface name="position">
-                <param name="min">-${PI/2}</param>
-                <param name="max">${PI/2}</param>
-            </command_interface>
-            <state_interface name="position"/>
-        </joint>
-    <!-- End of Griper -->
     </ros2_control>
 </robot>

Commit message: no gripper version

File: src/yaskawa_mh5_description/urdf/TesseraVue_3D_sensor_bigger.urdf.xacro (robot description, xacro)
@@ -37,5 +37,6 @@
     <parent link="tesseravue_chassis_link"/>
     <child link="tesseravue_camera_link"/>
-    <origin xyz="0.096 0.07 0.38" rpy="0 -1.5708 0"/>
+    <origin xyz="0.096 0.07 0.38" rpy="0 0 0"/>
+    <!-- 1.5708 -->
     <!-- <origin xyz="0.0765 0 0.06" rpy="0 0 0"/> Adjust as needed -->
   </joint>
@@ -53,12 +54,10 @@
     <parent link="tesseravue_camera_link"/>
     <child link="3dcamera_optical"/>
-    <origin xyz="0 0 0" rpy="0 0 0"/>
-    <!-- <origin xyz="0 0 0" rpy="-1.5708 0 -1.5708"/>  -->
-    <origin xyz="0 0 0" rpy="${-PI/2} 0 ${-PI/2}"/>
+    <origin xyz="0 0 0" rpy="${PI/2} 0 -${PI/2}"/>
   </joint>
   <link name="3dcamera_optical"/>
   <gazebo reference="tesseravue_camera_link">
     <sensor type="camera" name="TesseraVue">
-      <pose> 0 0 0 0 0 0 </pose>
+      <pose>0 0 0 0 0 0 </pose>
       <visualize>true</visualize>
       <update_rate>12.0</update_rate>
@@ -66,6 +65,6 @@
         <horizontal_fov>1.089</horizontal_fov>
         <image>
-          <width>800</width>
-          <height>800</height>
+          <width>1504</width>
+          <height>2048</height>
           <format>R8G8B8</format>
         </image>

File: src/yaskawa_mh5_description/urdf/mh5.urdf.xacro (robot description, xacro)
@@ -5,12 +5,8 @@
 <!-- =================================================================================== -->
 <robot name="yaskawa_mh5lf" xmlns:xacro="http://ros.org/wiki/xacro">
-  <xacro:include filename="$(find yaskawa_mh5_description)/urdf/mh5_gazebo.urdf.xacro"/>
+  <xacro:include filename="$(find yaskawa_mh5_description)/urdf/mh5_gazebo.xacro"/>
   <xacro:include filename="$(find yaskawa_mh5_description)/urdf/mh5_ros2_controller.urdf.xacro"/>
   <xacro:include filename="$(find yaskawa_mh5_description)/urdf/TesseraVue_3D_sensor_bigger.urdf.xacro"/>
-  <!-- <xacro:include filename="$(find yaskawa_mh5_description)/urdf/grippers.urdf.xacro"/> -->
 <!-- macro function for inertial-->
-  <xacro:property name="effort" value="30.0"/>
-  <xacro:property name="velocity" value="10.0"/>
-  <xacro:property name="PI" value="3.14159"/>
 	<xacro:macro name="default_inertial" params="mass">
 		<inertial>
@@ -21,5 +17,4 @@
 		</inertial>
 	</xacro:macro>
-<!-- end of macro function for inertial -->
 <!-- transmission for robot controller -->
   <xacro:macro name="default_transmission" params="number">
@@ -34,10 +29,9 @@
   </xacro:macro>
 <!-- end transmission for robot controller -->
-  <!-- link list -->
   <link name = "world" />
   <link name="base_link">
     <xacro:default_inertial mass="1.0"/>
     <visual>
-     <origin rpy="0 0 0"/>
+      <origin rpy="0 0 3.14159"/>
       <geometry>
         <mesh filename="package://yaskawa_mh5_description/meshes/mh5/visual/MH5_BASE_AXIS.stl" scale="2.0 2.0 2.0"/>
@@ -87,5 +81,5 @@
       </geometry>
       <material name="yellow"/>
-    </collision>
+      </collision>
   </link>
   <link name="link_u">
@@ -111,4 +105,19 @@
       </geometry>
       <material name="silver"/>
+    </visual>
+    <collision>
+      <geometry>
+        <mesh filename="package://yaskawa_mh5_description/meshes/mh5/collision/MH5_R_AXIS.stl" scale="2.0 2.0 2.0"/>
+      </geometry>
+      <material name="yellow"/>
+    </collision>
+  </link>
+  <link name="link_b">
+    <xacro:default_inertial mass="1.0"/>
+    <visual>
+      <geometry>
+        <mesh filename="package://yaskawa_mh5_description/meshes/mh5/visual/MH5_B_AXIS.stl" scale="2.0 2.0 2.0"/>
+      </geometry>
+      <material name="blue"/>
     </visual>
     <collision>
@@ -144,9 +153,9 @@
     <parent link="base_link"/>
     <child link="link_s"/>
-    <origin rpy="0 0 0" xyz="0 0 0.3980"/>
+    <origin rpy="0 0 0" xyz="0 0 0.1990"/>
     <axis xyz="0 0 1"/>
-    <limit effort="100" lower="-1.1345" upper="2.6180" velocity="2.96"/>
-  </joint>
-  <joint name="joint_l" type="revolute">
+    <limit effort="100" lower="-2.9671" upper="2.9671" velocity="2.96"/>
+  </joint>
+ <joint name="joint_l" type="revolute">
     <parent link="link_s"/>
     <child link="link_l"/>
@@ -176,5 +185,5 @@
     <limit effort="100" lower="-2.1817" upper="2.1817" velocity="3.48"/>
   </joint>
-  <joint name="joint_t" type="fixed">
+  <joint name="joint_t" type="revolute">
     <parent link="link_b"/>
     <child link="link_t"/>
@@ -190,4 +199,3 @@
     <xacro:default_transmission number="b"/>
     <xacro:default_transmission number="t"/>
-    <!-- <xacro:default_transmission number="a"/>  -->
 </robot>
