Commit message: robotiq_85 gripper is implemented

File: src/yaskawa_mh5_description/urdf/TesseraVue_3D_sensor_bigger.urdf.xacro (robot description, xacro)
@@ -15,5 +15,5 @@
     <parent link="link_r"/>
     <child link="tesseravue_chassis_link"/>
-    <origin xyz="0.0715 0.05 0.08" rpy="1.5708 0 1.5708"/> <!-- Adjust as needed -->
+    <origin xyz="0.0715 0.05 0.08" rpy="1.5708 0 1.5708"/>
   </joint>
   <!-- 3D sensor -->
@@ -27,4 +27,5 @@
     </visual>
     <collision>
+    <origin xyz="0 0.05 0.3" rpy="0 0 0"/>
       <geometry>
         <mesh filename="package://yaskawa_mh5_description/meshes/mh5/collision/BIN_PICKING_MODULE_1CH_ASM.stl" scale="0.0015 0.0015 0.0015"/>
@@ -37,5 +38,6 @@
     <parent link="tesseravue_chassis_link"/>
     <child link="tesseravue_camera_link"/>
-    <origin xyz="0.096 0.07 0.38" rpy="0 0 0"/>
+     <origin xyz="0.096 0.07 0.38" rpy="-${PI/2} -${PI/2} 0"/>
+    <!-- <origin xyz="0.096 0.07 0.38" rpy="${PI/2} 0 ${PI/2}"/> -->
     <!-- 1.5708 -->
     <!-- <origin xyz="0.0765 0 0.06" rpy="0 0 0"/> Adjust as needed -->
@@ -49,10 +51,16 @@
       <material name="blue"/>
     </visual>
+    <collision>
+    <geometry>
+        <cylinder radius = "0.0005" length = "0.001"/>
+      </geometry>
+    </collision>
   </link>
   <!-- Virtual link for optical joint -->
   <joint name="3dcamera_optical_joint" type="fixed">
-    <parent link="tesseravue_camera_link"/>
+    <parent link="tesseravue_camera_link"/>${PI/2}
     <child link="3dcamera_optical"/>
-    <origin xyz="0 0 0" rpy="${PI/2} 0 -${PI/2}"/>
+    <!-- <origin xyz="0 0 0" rpy="${PI/2} 0 -${PI/2}"/>  -->
+    <origin xyz="0 0 0" rpy="0 0 0"/>
   </joint>
   <link name="3dcamera_optical"/>
@@ -65,6 +73,6 @@
         <horizontal_fov>1.089</horizontal_fov>
         <image>
-          <width>1504</width>
-          <height>2048</height>
+          <width>3840</width>
+          <height>2160</height>
           <format>R8G8B8</format>
         </image>

File: src/yaskawa_mh5_description/urdf/mh5.urdf.xacro (robot description, xacro)
@@ -8,4 +8,5 @@
   <xacro:include filename="$(find yaskawa_mh5_description)/urdf/mh5_ros2_controller.urdf.xacro"/>
   <xacro:include filename="$(find yaskawa_mh5_description)/urdf/TesseraVue_3D_sensor_bigger.urdf.xacro"/>
+  <xacro:include filename="$(find yaskawa_mh5_description)/urdf/robotiq_85_gripper_macro.urdf.xacro"/>
 <!-- macro function for inertial-->
 	<xacro:macro name="default_inertial" params="mass">
@@ -153,5 +154,5 @@
     <parent link="base_link"/>
     <child link="link_s"/>
-    <origin rpy="0 0 0" xyz="0 0 0.1990"/>
+    <origin rpy="0 0 0" xyz="0 0 0.40"/>
     <axis xyz="0 0 1"/>
     <limit effort="100" lower="-2.9671" upper="2.9671" velocity="2.96"/>
@@ -183,12 +184,12 @@
     <origin rpy="0 0 0" xyz="0.4670 0 0"/>
     <axis xyz="0 -1 0"/>
-    <limit effort="100" lower="-2.1817" upper="2.1817" velocity="3.48"/>
-  </joint>
-  <joint name="joint_t" type="revolute">
-    <parent link="link_b"/>
-    <child link="link_t"/>
-    <origin rpy="0 0 0" xyz="0.1730 0 0"/>
-    <axis xyz="0 -1 0"/>
-    <limit effort="100" lower="-6.2831" upper="6.2831" velocity="6.97"/>
+    <limit effort="100" lower="-0.610865" upper="0.610865" velocity="6.97"/>
+  </joint>
+  <joint name="joint_t" type="continuous">
+      <parent link="link_b"/>
+      <child link="link_t"/>
+      <origin rpy="0 0 0" xyz="0.1730 0 0"/>
+      <axis xyz="1 0 0"/>
+      <limit effort="100" velocity="6.97"/>
   </joint>
   <!-- Define transmissions -->

File: src/yaskawa_mh5_description/urdf/mh5_gazebo.xacro (robot description, xacro)
@@ -1,4 +1,5 @@
 <?xml version="1.0"?>
 <robot xmlns:xacro="http://ros.org/wiki/xacro" name="yaskawa_mh5lf">
+ <xacro:property name="PI" value="3.14159"/>
     <gazebo>
         <plugin filename="libgazebo_ros2_control.so" name="gazebo_ros2_control">
@@ -7,4 +8,37 @@
             <parameters>$(find yaskawa_mh5_controller)/config/mh5_ros2_controller.yaml</parameters>
         </plugin>
+            <plugin filename="libroboticsgroup_upatras_gazebo_mimic_joint_plugin.so" name="mimic_robotiq_85_1">
+                <joint>robotiq_85_left_knuckle_joint</joint>
+                <mimicJoint>robotiq_85_right_knuckle_joint</mimicJoint>
+                <!--multiplier>1.0</multiplier>
+                <offset>0.0</offset-->                 <command_interface name="position">
+                    <param name="min">-${PI/2}</param>
+                    <param name="max">${PI/2}</param>
+                </command_interface>
+            </plugin>
+            <plugin filename="libroboticsgroup_upatras_gazebo_mimic_joint_plugin.so" name="mimic_robotiq_85_2">
+                <joint>robotiq_85_left_knuckle_joint</joint>
+                <mimicJoint>robotiq_85_left_inner_knuckle_joint</mimicJoint>
+                <!--multiplier>1.0</multiplier>
+                <offset>0.0</offset-->
+            </plugin>
+            <plugin filename="libroboticsgroup_upatras_gazebo_mimic_joint_plugin.so" name="mimic_robotiq_85_3">
+                <joint>robotiq_85_left_knuckle_joint</joint>
+                <mimicJoint>robotiq_85_right_inner_knuckle_joint</mimicJoint>
+                <!--multiplier>1.0</multiplier>
+                <offset>0.0</offset-->
+            </plugin>
+            <plugin filename="libroboticsgroup_upatras_gazebo_mimic_joint_plugin.so" name="mimic_robotiq_85_4">
+                <joint>robotiq_85_left_knuckle_joint</joint>
+                <mimicJoint>robotiq_85_left_finger_tip_joint</mimicJoint>
+                <multiplier>-1.0</multiplier>
+                <!--offset>0.0</offset-->
+            </plugin>
+            <plugin filename="libroboticsgroup_upatras_gazebo_mimic_joint_plugin.so" name="mimic_robotiq_85_5">
+                <joint>robotiq_85_left_knuckle_joint</joint>
+                <mimicJoint>robotiq_85_right_finger_tip_joint</mimicJoint>
+                <multiplier>-1.0</multiplier>
+                <!--offset>0.0</offset-->
+            </plugin>
     </gazebo>
 </robot>

File: src/yaskawa_mh5_description/urdf/mh5_ros2_controller.urdf.xacro (robot description, xacro)
@@ -2,9 +2,9 @@
 <robot xmlns:xacro="http://ros.org/wiki/xacro" name="yaskawa_mh5lf">
     <xacro:property name="PI" value="3.14159"/>
-    <!-- <xacro:include filename="$(find yaskawa_mh5_description)/urdf/robotiq_85_gripper.transmission.xacro"/> -->
     <ros2_control name="RobotSystem" type="system">
         <hardware>
             <plugin>gazebo_ros2_control/GazeboSystem</plugin>
         </hardware>
+        <!-- Robot Arm Joints -->
         <joint name="joint_s">
             <command_interface name="position">
@@ -14,5 +14,5 @@
             <state_interface name="position"/>
         </joint>
-        <joint name="joint_l"><xacro:property name="PI" value="3.14159"/>
+        <joint name="joint_l">
             <command_interface name="position">
                 <param name="min">-${PI/2}</param>
@@ -23,5 +23,5 @@
         <joint name="joint_u">
             <command_interface name="position">
-                <param name="min">-${PI/2}</param><xacro:property name="PI" value="3.14159"/>
+                <param name="min">-${PI/2}</param>
                 <param name="max">${PI/2}</param>
             </command_interface>
@@ -49,4 +49,56 @@
             <state_interface name="position"/>
         </joint>
+        <!-- Gripper Joints -->
+        <joint name="robotiq_85_left_knuckle_joint">
+                <param name="min">-${PI/2}</param>
+                <param name="max">${PI/2}</param>
+            <command_interface name="position" />
+            <state_interface name="position"/>
+        </joint>
+        <joint name="robotiq_85_right_knuckle_joint">
+            <param name="mimic">robotiq_85_left_knuckle_joint</param>
+            <param name="multiplier">1</param>
+             <command_interface name="position">
+                <param name="min">-${PI/2}</param>
+                <param name="max">${PI/2}</param>
+            </command_interface>
+            <state_interface name="position"/>
+        </joint>
+        <joint name="robotiq_85_left_inner_knuckle_joint">
+            <param name="mimic">robotiq_85_left_knuckle_joint</param>
+            <param name="multiplier">1</param>
+           <command_interface name="position">
+                <param name="min">-${PI/2}</param>
+                <param name="max">${PI/2}</param>
+            </command_interface>
+            <state_interface name="position"/>
+        </joint>
+        <joint name="robotiq_85_right_inner_knuckle_joint">
+            <param name="mimic">robotiq_85_left_knuckle_joint</param>
+            <param name="multiplier">1</param>
+            <command_interface name="position">
+                <param name="min">-${PI/2}</param>
+                <param name="max">${PI/2}</param>
+            </command_interface>
+            <state_interface name="position"/>
+        </joint>
+        <joint name="robotiq_85_left_finger_tip_joint">
+            <param name="mimic">robotiq_85_left_knuckle_joint</param>
+            <param name="multiplier">-1</param>
+            <command_interface name="position">
+                <param name="min">-${PI/2}</param>
+                <param name="max">${PI/2}</param>
+            </command_interface>
+            <state_interface name="position"/>
+        </joint>
+        <joint name="robotiq_85_right_finger_tip_joint">
+            <param name="mimic">robotiq_85_left_knuckle_joint</param>
+            <param name="multiplier">-1</param>
+            <command_interface name="position">
+                <param name="min">-${PI/2}</param>
+                <param name="max">${PI/2}</param>
+            </command_interface>
+            <state_interface name="position"/>
+        </joint>
     </ros2_control>
 </robot>

Commit message: Camera is fixed on teh Pole

File: src/yaskawa_mh5_description/urdf/TesseraVue_3D_sensor_bigger.urdf.xacro (robot description, xacro)
@@ -13,7 +13,7 @@
   <!-- TesseraVue Visualization on Gazebo -->
   <joint name="tesseravue_chassis_joint" type="fixed">
-    <parent link="link_r"/>
+    <parent link="world"/>
     <child link="tesseravue_chassis_link"/>
-    <origin xyz="0.0715 0.05 0.08" rpy="1.5708 0 1.5708"/>
+    <origin xyz="3 0 0" rpy="0 0 -1.5708"/>
   </joint>
   <!-- 3D sensor -->
@@ -21,13 +21,13 @@
     <xacro:default_inertial mass="0.5"/>
     <visual>
-    <origin xyz="0 0.05 0.3" rpy="0 0 0"/>
+    <origin xyz="0 0 0" rpy="0 0 0"/>
       <geometry>
-        <mesh filename="package://yaskawa_mh5_description/meshes/mh5/collision/BIN_PICKING_MODULE_1CH_ASM.stl" scale="0.0015 0.0015 0.0015"/>
+        <mesh filename="package://yaskawa_mh5_description/meshes/mh5/collision/tessaraVue_with_pole.stl" scale="0.04 0.04 0.04"/>
       </geometry>
     </visual>
     <collision>
-    <origin xyz="0 0.05 0.3" rpy="0 0 0"/>
+    <origin xyz="0 0 0" rpy="0 0 0"/>
       <geometry>
-        <mesh filename="package://yaskawa_mh5_description/meshes/mh5/collision/BIN_PICKING_MODULE_1CH_ASM.stl" scale="0.0015 0.0015 0.0015"/>
+        <mesh filename="package://yaskawa_mh5_description/meshes/mh5/collision/tessaraVue_with_pole.stl" scale="0.04 0.04 0.04"/>
       </geometry>
     </collision>
@@ -38,5 +38,5 @@
     <parent link="tesseravue_chassis_link"/>
     <child link="tesseravue_camera_link"/>
-     <origin xyz="0.096 0.07 0.38" rpy="-${PI/2} -${PI/2} 0"/>
+     <origin xyz="0.096 -0.15   1.5" rpy="0 ${PI/5} -${PI/2}"/>
     <!-- <origin xyz="0.096 0.07 0.38" rpy="${PI/2} 0 ${PI/2}"/> -->
     <!-- 1.5708 -->
@@ -59,8 +59,8 @@
   <!-- Virtual link for optical joint -->
   <joint name="3dcamera_optical_joint" type="fixed">
-    <parent link="tesseravue_camera_link"/>${PI/2}
+    <parent link="tesseravue_camera_link"/>
     <child link="3dcamera_optical"/>
-    <!-- <origin xyz="0 0 0" rpy="${PI/2} 0 -${PI/2}"/>  -->
-    <origin xyz="0 0 0" rpy="0 0 0"/>
+    <origin xyz="0 0 0" rpy="${PI/2} 0 -${PI/2}"/>
+    <!-- <origin xyz="0 0 0" rpy="0 0 0"/>  -->
   </joint>
   <link name="3dcamera_optical"/>

File: src/yaskawa_mh5_description/urdf/mh5.urdf.xacro (robot description, xacro)
@@ -87,4 +87,5 @@
     <xacro:default_inertial mass="1.0"/>
     <visual>
+p
       <geometry>
         <mesh filename="package://yaskawa_mh5_description/meshes/mh5/visual/MH5_U_AXIS.stl" scale="2.0 2.0 2.0"/>
@@ -179,4 +180,5 @@
     <limit effort="100" lower="-3.3161" upper="3.3161" velocity="3.48"/>
   </joint>
+allow-overriding yaskawa_mh5_description
   <joint name="joint_b" type="revolute">
     <parent link="link_r"/>

Commit message: 3d sensor in pole

File: src/yaskawa_mh5_description/urdf/TesseraVue_3D_sensor_bigger.urdf.xacro (robot description, xacro)
@@ -15,5 +15,5 @@
     <parent link="world"/>
     <child link="tesseravue_chassis_link"/>
-    <origin xyz="3 0 0" rpy="0 0 -1.5708"/>
+    <origin xyz="2.5 0 0" rpy="0 0 -1.5708"/>
   </joint>
   <!-- 3D sensor -->
@@ -38,5 +38,5 @@
     <parent link="tesseravue_chassis_link"/>
     <child link="tesseravue_camera_link"/>
-     <origin xyz="0.096 -0.15   1.5" rpy="0 ${PI/5} -${PI/2}"/>
+     <origin xyz="0.096 -0.15   1.5" rpy="0 ${PI/4} -${PI/2}"/>
     <!-- <origin xyz="0.096 0.07 0.38" rpy="${PI/2} 0 ${PI/2}"/> -->
     <!-- 1.5708 -->
@@ -69,15 +69,15 @@
       <pose>0 0 0 0 0 0 </pose>
       <visualize>true</visualize>
-      <update_rate>12.0</update_rate>
+      <update_rate>5.0</update_rate>
       <camera name="TesseraVue">
         <horizontal_fov>1.089</horizontal_fov>
         <image>
           <width>3840</width>
-          <height>2160</height>
+          <height>5840</height>
           <format>R8G8B8</format>
         </image>
         <clip>
-          <near>0.05</near>
-          <far>8.0</far>
+          <near>0.5</near>
+          <far>20.0</far>
         </clip>
       </camera>

File: src/yaskawa_mh5_description/urdf/robotiq_85_gripper_macro.urdf.xacro (robot description, xacro)
@@ -286,4 +286,29 @@
 		</gazebo>
 		<xacro:robotiq_85_gripper_transmission />
+		<joint name="robotiq_85_left_finger_tip_joint_mimic" type="fixed">
+			<parent link="world" />
+			<child link="random" />
+		</joint>
+		<link name="random"/>
+		<joint name="robotiq_85_right_finger_tip_joint_mimic" type="fixed">
+			<parent link="world" />
+			<child link="random2" />
+		</joint>
+		<link name="random2"/>
+		<joint name="robotiq_85_right_inner_knuckle_joint_mimic" type="fixed">
+			<parent link="world" />
+			<child link="random3" />
+		</joint>
+				<link name="random3"/>
+		<joint name="robotiq_85_left_inner_knuckle_joint_mimic" type="fixed">
+			<parent link="world" />
+			<child link="random4" />
+		</joint>
+		<link name="random4"/>
+		<joint name="robotiq_85_right_knuckle_joint_mimic" type="fixed">
+			<parent link="world" />
+			<child link="random5" />
+		</joint>
+		<link name="random5"/>
 	<!-- </xacro:macro> -->
 </robot>
