Commit message: grasp planning and cartesion planning is done

File: src/yaskawa_mh5_description/urdf/TesseraVue_3D_sensor_bigger.urdf.xacro (robot description, xacro)
@@ -15,5 +15,5 @@
     <parent link="world"/>
     <child link="tesseravue_chassis_link"/>
-    <origin xyz="2.5 0 0" rpy="0 0 -1.5708"/>
+    <origin xyz="0 -2 0" rpy="0 0 2.5708"/>
   </joint>
   <!-- 3D sensor -->

File: src/yaskawa_mh5_description/urdf/mh5.urdf.xacro (robot description, xacro)
@@ -1,12 +1,10 @@
 <?xml version="1.0" ?>
-<!-- =================================================================================== -->
-<!-- |    This document was autogenerated by xacro from mh5.xacro                      | -->
-<!-- |    EDITING THIS FILE BY HAND IS NOT RECOMMENDED                                 | -->
-<!-- =================================================================================== -->
 <robot name="yaskawa_mh5lf" xmlns:xacro="http://ros.org/wiki/xacro">
   <xacro:include filename="$(find yaskawa_mh5_description)/urdf/mh5_gazebo.xacro"/>
+  <!-- <xacro:include filename="$(find yaskawa_mh5_description)/urdf/robotiq_85_gripper.ros2_control.xacro"/> -->
   <xacro:include filename="$(find yaskawa_mh5_description)/urdf/mh5_ros2_controller.urdf.xacro"/>
   <xacro:include filename="$(find yaskawa_mh5_description)/urdf/TesseraVue_3D_sensor_bigger.urdf.xacro"/>
-  <xacro:include filename="$(find yaskawa_mh5_description)/urdf/robotiq_85_gripper_macro.urdf.xacro"/>
+  <xacro:include filename="$(find yaskawa_mh5_description)/urdf/robotiq_85_gripper.urdf.xacro"/>
+  <!-- <xacro:include filename="$(find point_cloud_processing)/urdf/dynamic_object.urdf.xacro"/> -->
 <!-- macro function for inertial-->
 	<xacro:macro name="default_inertial" params="mass">
@@ -164,5 +162,5 @@
     <origin rpy="0 0 0" xyz="0.1760 0 0.2620"/>
     <axis xyz="0 1 0"/>
-    <limit effort="100" lower="-1.1345" upper="2.6180" velocity="2.96"/>
+    <limit effort="100" lower="-1" upper="2.0" velocity="2.96"/>
   </joint>
   <joint name="joint_u" type="revolute">
@@ -171,5 +169,5 @@
     <origin rpy="0 0 0" xyz="0 0 0.6200"/>
     <axis xyz="0 -1 0"/>
-    <limit effort="100" lower="-1.0122" upper="3.2218" velocity="2.96"/>
+    <limit effort="100" lower="-0.22" upper="1.5" velocity="2.96"/>
   </joint>
   <joint name="joint_r" type="revolute">
@@ -185,5 +183,5 @@
     <origin rpy="0 0 0" xyz="0.4670 0 0"/>
     <axis xyz="0 -1 0"/>
-    <limit effort="100" lower="-0.610865" upper="0.610865" velocity="6.97"/>
+    <limit effort="100" lower="-0.610865" upper="1.610865" velocity="6.97"/>
   </joint>
   <joint name="joint_t" type="continuous">

File: src/yaskawa_mh5_description/urdf/mh5_gazebo.xacro (robot description, xacro)
@@ -8,37 +8,4 @@
             <parameters>$(find yaskawa_mh5_controller)/config/mh5_ros2_controller.yaml</parameters>
         </plugin>
-            <plugin filename="libroboticsgroup_upatras_gazebo_mimic_joint_plugin.so" name="mimic_robotiq_85_1">
-                <joint>robotiq_85_left_knuckle_joint</joint>
-                <mimicJoint>robotiq_85_right_knuckle_joint</mimicJoint>
-                <!--multiplier>1.0</multiplier>
-                <offset>0.0</offset-->                 <command_interface name="position">
-                    <param name="min">-${PI/2}</param>
-                    <param name="max">${PI/2}</param>
-                </command_interface>
-            </plugin>
-            <plugin filename="libroboticsgroup_upatras_gazebo_mimic_joint_plugin.so" name="mimic_robotiq_85_2">
-                <joint>robotiq_85_left_knuckle_joint</joint>
-                <mimicJoint>robotiq_85_left_inner_knuckle_joint</mimicJoint>
-                <!--multiplier>1.0</multiplier>
-                <offset>0.0</offset-->
-            </plugin>
-            <plugin filename="libroboticsgroup_upatras_gazebo_mimic_joint_plugin.so" name="mimic_robotiq_85_3">
-                <joint>robotiq_85_left_knuckle_joint</joint>
-                <mimicJoint>robotiq_85_right_inner_knuckle_joint</mimicJoint>
-                <!--multiplier>1.0</multiplier>
-                <offset>0.0</offset-->
-            </plugin>
-            <plugin filename="libroboticsgroup_upatras_gazebo_mimic_joint_plugin.so" name="mimic_robotiq_85_4">
-                <joint>robotiq_85_left_knuckle_joint</joint>
-                <mimicJoint>robotiq_85_left_finger_tip_joint</mimicJoint>
-                <multiplier>-1.0</multiplier>
-                <!--offset>0.0</offset-->
-            </plugin>
-            <plugin filename="libroboticsgroup_upatras_gazebo_mimic_joint_plugin.so" name="mimic_robotiq_85_5">
-                <joint>robotiq_85_left_knuckle_joint</joint>
-                <mimicJoint>robotiq_85_right_finger_tip_joint</mimicJoint>
-                <multiplier>-1.0</multiplier>
-                <!--offset>0.0</offset-->
-            </plugin>
     </gazebo>
 </robot>

File: src/yaskawa_mh5_description/urdf/mh5_ros2_controller.urdf.xacro (robot description, xacro)
@@ -3,4 +3,5 @@
     <xacro:property name="PI" value="3.14159"/>
     <ros2_control name="RobotSystem" type="system">
+    <!-- <xacro:include filename="$(find yaskawa_mh5_description)/urdf/robotiq_85_gripper.ros2_control.xacro"/> -->
         <hardware>
             <plugin>gazebo_ros2_control/GazeboSystem</plugin>
@@ -12,6 +13,6 @@
                 <param name="max">${PI/2}</param>
             </command_interface>
-            <state_interface name="position"/>
-        </joint>
+             <state_interface name="position"/>
+             </joint>
         <joint name="joint_l">
             <command_interface name="position">
@@ -49,56 +50,45 @@
             <state_interface name="position"/>
         </joint>
-        <!-- Gripper Joints -->
         <joint name="robotiq_85_left_knuckle_joint">
-                <param name="min">-${PI/2}</param>
-                <param name="max">${PI/2}</param>
-            <command_interface name="position" />
-            <state_interface name="position"/>
-        </joint>
-        <joint name="robotiq_85_right_knuckle_joint">
-            <param name="mimic">robotiq_85_left_knuckle_joint</param>
-            <param name="multiplier">1</param>
-             <command_interface name="position">
-                <param name="min">-${PI/2}</param>
-                <param name="max">${PI/2}</param>
-            </command_interface>
-            <state_interface name="position"/>
-        </joint>
-        <joint name="robotiq_85_left_inner_knuckle_joint">
-            <param name="mimic">robotiq_85_left_knuckle_joint</param>
-            <param name="multiplier">1</param>
-           <command_interface name="position">
-                <param name="min">-${PI/2}</param>
-                <param name="max">${PI/2}</param>
-            </command_interface>
-            <state_interface name="position"/>
-        </joint>
-        <joint name="robotiq_85_right_inner_knuckle_joint">
-            <param name="mimic">robotiq_85_left_knuckle_joint</param>
-            <param name="multiplier">1</param>
-            <command_interface name="position">
-                <param name="min">-${PI/2}</param>
-                <param name="max">${PI/2}</param>
-            </command_interface>
-            <state_interface name="position"/>
-        </joint>
-        <joint name="robotiq_85_left_finger_tip_joint">
-            <param name="mimic">robotiq_85_left_knuckle_joint</param>
-            <param name="multiplier">-1</param>
-            <command_interface name="position">
-                <param name="min">-${PI/2}</param>
-                <param name="max">${PI/2}</param>
-            </command_interface>
-            <state_interface name="position"/>
-        </joint>
-        <joint name="robotiq_85_right_finger_tip_joint">
-            <param name="mimic">robotiq_85_left_knuckle_joint</param>
-            <param name="multiplier">-1</param>
-            <command_interface name="position">
-                <param name="min">-${PI/2}</param>
-                <param name="max">${PI/2}</param>
-            </command_interface>
-            <state_interface name="position"/>
-        </joint>
+                <param name="initial_position">0.7929</param>
+                <command_interface name="position" />
+                <state_interface name="position"/>
+                <state_interface name="velocity"/>
+            </joint>
+            <joint name="robotiq_85_right_knuckle_joint">
+                <param name="mimic">robotiq_85_left_knuckle_joint</param>
+                <param name="multiplier">1</param>
+                <command_interface name="position" />
+                <state_interface name="position"/>
+                <state_interface name="velocity"/>
+            </joint>
+            <joint name="robotiq_85_left_inner_knuckle_joint">
+                <param name="mimic">robotiq_85_left_knuckle_joint</param>
+                <param name="multiplier">1</param>
+                <command_interface name="position" />
+                <state_interface name="position"/>
+                <state_interface name="velocity"/>
+            </joint>
+            <joint name="robotiq_85_right_inner_knuckle_joint">
+                <param name="mimic">robotiq_85_left_knuckle_joint</param>
+                <param name="multiplier">1</param>
+                <command_interface name="position" />
+                <state_interface name="position"/>
+                <state_interface name="velocity"/>
+            </joint>
+            <joint name="robotiq_85_left_finger_tip_joint">
+                <param name="mimic">robotiq_85_left_knuckle_joint</param>
+                <param name="multiplier">-1</param>
+                <command_interface name="position" />
+                <state_interface name="position"/>
+                <state_interface name="velocity"/>
+            </joint>
+            <joint name="robotiq_85_right_finger_tip_joint">
+                <param name="mimic">robotiq_85_left_knuckle_joint</param>
+                <param name="multiplier">-1</param>
+                <command_interface name="position" />
+                <state_interface name="position"/>
+                <state_interface name="velocity"/>
+            </joint>
     </ros2_control>
 </robot>

File: src/yaskawa_mh5_description/urdf/robotiq_85_gripper.transmission.xacro (robot description, xacro)
@@ -1,48 +1,66 @@
 <?xml version="1.0"?>
 <robot xmlns:xacro="http://ros.org/wiki/xacro">
-  <xacro:macro name="robotiq_85_gripper_transmission">
-        <transmission name="robotiq_85_left_knuckle_trans">
+  <xacro:macro name="robotiq_85_gripper_transmission" params="prefix">
+        <!-- <transmission name="${prefix}robotiq_85_left_knuckle_trans">
             <type>transmission_interface/SimpleTransmission</type>
-            <joint name="finger_joint">
+            <joint name="${prefix}robotiq_85_left_knuckle_joint">
                 <hardwareInterface>hardware_interface/PositionJointInterface</hardwareInterface>
             </joint>
-            <actuator name="robotiq_85_left_knuckle_motor">
+            <actuator name="${prefix}robotiq_85_left_knuckle_motor">
                 <mechanicalReduction>1</mechanicalReduction>
                 <hardwareInterface>hardware_interface/PositionJointInterface</hardwareInterface>
             </actuator>
+        </transmission> -->
+        <transmission name="${prefix}robotiq_85_left_knuckle_trans">
+            <type>transmission_interface/SimpleTransmission</type>
+            <joint name="${prefix}robotiq_85_left_knuckle_joint">
+                <hardwareInterface>hardware_interface/EffortJointInterface</hardwareInterface>
+            </joint>
+            <actuator name="${prefix}robotiq_85_left_knuckle_motor">
+                <mechanicalReduction>1</mechanicalReduction>
+                <hardwareInterface>hardware_interface/EffortJointInterface</hardwareInterface>
+            </actuator>
         </transmission>
         <gazebo>
-            <plugin filename="libroboticsgroup_gazebo_mimic_joint_plugin.so" name="mimic_robotiq_85_1">
-                <joint>finger_joint</joint>
-                <mimicJoint>left_inner_knuckle_joint</mimicJoint>
-                <!--multiplier>1.0</multiplier>
-                <offset>0.0</offset-->
+                <!-- loading plugin mimic joints works in gazebo now -->
+            <plugin filename="libroboticsgroup_gazebo_mimic_joint_plugin.so" name="${prefix}mimic_robotiq_85_1">
+                <joint>${prefix}robotiq_85_left_knuckle_joint</joint>
+                <mimicJoint>${prefix}robotiq_85_right_knuckle_joint</mimicJoint>
+                <multiplier>1.0</multiplier>
+                <offset>0.0</offset>
             </plugin>
-            <plugin filename="libroboticsgroup_gazebo_mimic_joint_plugin.so" name="mimic_robotiq_85_2">
-                <joint>finger_joint</joint>
-                <mimicJoint>left_inner_finger_joint</mimicJoint>
-                <!--multiplier>1.0</multiplier>
-                <offset>0.0</offset-->
+            <plugin filename="libroboticsgroup_gazebo_mimic_joint_plugin.so" name="${prefix}mimic_robotiq_85_2">
+                <joint>${prefix}robotiq_85_left_knuckle_joint</joint>
+                <mimicJoint>${prefix}robotiq_85_left_inner_knuckle_joint</mimicJoint>
+                <multiplier>1.0</multiplier>
+                <offset>0.0</offset>
             </plugin>
-            <plugin filename="libroboticsgroup_gazebo_mimic_joint_plugin.so" name="mimic_robotiq_85_3">
-                <joint>finger_joint</joint>
-                <mimicJoint>right_inner_knuckle_joint</mimicJoint>
-                <!-- multiplier>1.0</multiplier>
-                <offset>0.0</offset-->
+            <plugin filename="libroboticsgroup_gazebo_mimic_joint_plugin.so" name="${prefix}mimic_robotiq_85_3">
+                <joint>${prefix}robotiq_85_left_knuckle_joint</joint>
+                <mimicJoint>${prefix}robotiq_85_right_inner_knuckle_joint</mimicJoint>
+                <multiplier>1.0</multiplier>
+                <offset>0.0</offset>
             </plugin>
-            <plugin filename="libroboticsgroup_gazebo_mimic_joint_plugin.so" name="mimic_robotiq_85_4">
-                <joint>finger_joint</joint>
-                <mimicJoint>right_inner_finger_joint</mimicJoint>
+            <plugin filename="libroboticsgroup_gazebo_mimic_joint_plugin.so" name="${prefix}mimic_robotiq_85_4">
+                <joint>${prefix}robotiq_85_left_knuckle_joint</joint>
+                <mimicJoint>${prefix}robotiq_85_left_finger_tip_joint</mimicJoint>
                 <multiplier>-1.0</multiplier>
                 <offset>0.0</offset>
             </plugin>
-            <plugin filename="libroboticsgroup_gazebo_mimic_joint_plugin.so" name="mimic_robotiq_85_5">
-                <joint>finger_joint</joint>
-                <mimicJoint>right_outer_knuckle_joint</mimicJoint>
+            <plugin filename="libroboticsgroup_gazebo_mimic_joint_plugin.so" name="${prefix}mimic_robotiq_85_5">
+                <joint>${prefix}robotiq_85_left_knuckle_joint</joint>
+                <mimicJoint>${prefix}robotiq_85_right_finger_tip_joint</mimicJoint>
                 <multiplier>-1.0</multiplier>
                 <offset>0.0</offset>
             </plugin>
+            <!-- <plugin name="gripper_control" filename="libgazebo_ros_joint_force_controller.so">
+                <joint>robotiq_85_left_knuckle_joint</joint>
+                <pid>100.0 0.01 10.0</pid>
+            </plugin> -->
+            <!-- <plugin name="gripper_control_right" filename="libgazebo_ros_joint_force_controller.so">
+                <joint>robotiq_85_right_knuckle_joint</joint>
+                <pid>100.0 0.01 10.0</pid>
+            </plugin>  -->
         </gazebo>
-         <!-- Define the mimic joints explicitly -->
     </xacro:macro>
 </robot>
