Commit message: grasp planning and cartesion planning is done

File: src/yaskawa_mh5_description/urdf/robotiq_85_gripper_macro.urdf.xacro (robot description, xacro)
@@ -2,11 +2,41 @@
 <robot xmlns:xacro="http://ros.org/wiki/xacro">
 	<xacro:include filename="$(find yaskawa_mh5_description)/urdf/robotiq_85_gripper.transmission.xacro" />
-	<!-- <xacro:macro name="robotiq_85_gripper" params="parent *origin sim:=false"> -->
-		<joint name="robotiq_85_base_joint" type="fixed">
-			<parent link="link_t"/>
-			<child link="robotiq_85_base_link"/>
-			<!-- <xacro:insert_block name="origin"/> -->
-		</joint>
-		<link name="robotiq_85_base_link">
+	<!-- <xacro:include filename="$(find yaskawa_mh5_description)/urdf/robotiq_85_gripper.transmission.effort.xacro" /> -->
+	<xacro:property name="PI" value="3.14159"/>
+	<xacro:macro name="mimic_joint_plugin_gazebo" params="name_prefix parent_joint mimic_joint has_pid:=false multiplier:=1.0 offset:=0 sensitiveness:=0.0 max_effort:=1.0 robot_namespace:=''">
+		<gazebo>
+			<plugin name="${name_prefix}mimic_joint_plugin" filename="libroboticsgroup_gazebo_mimic_joint_plugin.so">
+				<joint>${parent_joint}</joint>
+				<mimicJoint>${mimic_joint}</mimicJoint>
+				<xacro:if value="${has_pid}">
+					<hasPID />
+				</xacro:if>
+				<multiplier>${multiplier}</multiplier>
+				<offset>${offset}</offset>
+				<sensitiveness>${sensitiveness}</sensitiveness>
+				<maxEffort>${max_effort}</maxEffort>
+				<xacro:unless value="${robot_namespace == ''}">
+					<robotNamespace>($robot_namespace)</robotNamespace>
+				</xacro:unless>
+			</plugin>
+		</gazebo>
+	</xacro:macro>
+		<xacro:macro name="robotiq_85_gripper" params="prefix parent *origin sim:=false">
+		<!-- The current hardware driver does not depend on ros2_control but we do utilize
+				 it for simulating the gripper in Gazebo. Enabling this on hardware causes the
+				 JointStateBroadcaster to publish values for all joints including ones that are
+				 mimic'd which is causing issues on systems consuming the joint_state data. -->
+		<xacro:if value="${sim}">
+			<!-- ros2 control include -->
+			<xacro:include filename="$(find yaskawa_mh5_description)/urdf/robotiq_85_gripper.ros2_control.xacro"/>
+			<!-- ros2 control instance -->
+			<xacro:robotiq_85_gripper_ros2_control name="RobotiqGripperSystem"/>
+		</xacro:if>
+		<joint name="${prefix}robotiq_85_base_joint" type="fixed">
+			<parent link="${parent}"/>
+			<child link="${prefix}robotiq_85_base_link"/>
+			<xacro:insert_block name="origin"/>
+		</joint>
+		<link name="${prefix}robotiq_85_base_link">
 			<!-- Visual aid for grasping -->
 			<visual>
@@ -38,13 +68,13 @@
 			</inertial>
 		</link>
-		<joint name="robotiq_85_left_knuckle_joint" type="revolute">
-			<parent link="robotiq_85_base_link"/>
-			<child link="robotiq_85_left_knuckle_link"/>
-			<axis xyz="0 0 1"/>
-			<origin rpy="${pi} 0.0 0.0" xyz="0.05490451627 0.03060114443 0.0"/>
+		<joint name="${prefix}robotiq_85_left_knuckle_joint" type="revolute">
+			<parent link="${prefix}robotiq_85_base_link"/>
+			<child link="${prefix}robotiq_85_left_knuckle_link"/>
+			<axis xyz="0 0 1"/>
+			<origin rpy="${PI} 0.0 0.0" xyz="0.05490451627 0.03060114443 0.0"/>
 			<limit lower="0.0" upper="0.804" velocity="0.5" effort="50"/>
 			<dynamics damping="100.0" />
 		</joint>
-		<gazebo reference="robotiq_85_left_knuckle_link">
+		<gazebo reference="${prefix}robotiq_85_left_knuckle_link">
 			<kp>1000000.0</kp>
 			<kd>100.0</kd>
@@ -55,14 +85,14 @@
 			<material>Gazebo/Grey</material>
 		</gazebo>
-		<joint name="robotiq_85_right_knuckle_joint" type="continuous">
-			<parent link="robotiq_85_base_link"/>
-			<child link="robotiq_85_right_knuckle_link"/>
+		<joint name="${prefix}robotiq_85_right_knuckle_joint" type="continuous">
+			<parent link="${prefix}robotiq_85_base_link"/>
+			<child link="${prefix}robotiq_85_right_knuckle_link"/>
 			<axis xyz="0 0 1"/>
 			<origin rpy="0.0 0.0 0.0" xyz="0.05490451627 -0.03060114443 0.0"/>
 			<limit lower="-3.14" upper="3.14" velocity="100.0" effort="50"/>
-			<mimic joint="robotiq_85_left_knuckle_joint"/>
+			<mimic joint="${prefix}robotiq_85_left_knuckle_joint"/>
 			<dynamics damping="100.0" />
 		</joint>
-		<gazebo reference="robotiq_85_right_knuckle_link">
+		<gazebo reference="${prefix}robotiq_85_right_knuckle_link">
 			<kp>1000000.0</kp>
 			<kd>100.0</kd>
@@ -73,5 +103,8 @@
 			<material>Gazebo/Grey</material>
 		</gazebo>
-		<link name="robotiq_85_left_knuckle_link">
+		<xacro:mimic_joint_plugin_gazebo name_prefix="{prefix}robotiq_85_right_knuckle_joint"
+			parent_joint="${prefix}robotiq_85_left_knuckle_joint" mimic_joint="${prefix}robotiq_85_right_knuckle_joint"
+			multiplier="1.0" max_effort="10.0" />
+		<link name="${prefix}robotiq_85_left_knuckle_link">
 			<visual>
 				<geometry>
@@ -92,5 +125,5 @@
 			</inertial>
 		</link>
-		<link name="robotiq_85_right_knuckle_link">
+		<link name="${prefix}robotiq_85_right_knuckle_link">
 			<visual>
 				<geometry>
@@ -111,15 +144,15 @@
 			</inertial>
 		</link>
-		<joint name="robotiq_85_left_finger_joint" type="fixed">
-			<parent link="robotiq_85_left_knuckle_link"/>
-			<child link="robotiq_85_left_finger_link"/>
+		<joint name="${prefix}robotiq_85_left_finger_joint" type="fixed">
+			<parent link="${prefix}robotiq_85_left_knuckle_link"/>
+			<child link="${prefix}robotiq_85_left_finger_link"/>
 			<origin xyz="-0.00408552455 -0.03148604435 0.0" rpy="0 0 0" />
 		</joint>
-		<joint name="robotiq_85_right_finger_joint" type="fixed">
-			<parent link="robotiq_85_right_knuckle_link"/>
-			<child link="robotiq_85_right_finger_link"/>
+		<joint name="${prefix}robotiq_85_right_finger_joint" type="fixed">
+			<parent link="${prefix}robotiq_85_right_knuckle_link"/>
+			<child link="${prefix}robotiq_85_right_finger_link"/>
 			<origin xyz="-0.00408552455 -0.03148604435 0.0" rpy="0 0 0" />
 		</joint>
-		<link name="robotiq_85_left_finger_link">
+		<link name="${prefix}robotiq_85_left_finger_link">
 			<visual>
 				<geometry>
@@ -140,5 +173,5 @@
 			</inertial>
 		</link>
-		<link name="robotiq_85_right_finger_link">
+		<link name="${prefix}robotiq_85_right_finger_link">
 			<visual>
 				<geometry>
@@ -159,21 +192,27 @@
 			</inertial>
 		</link>
-		<joint name="robotiq_85_left_inner_knuckle_joint" type="continuous">
-			<parent link="robotiq_85_base_link"/>
-			<child link="robotiq_85_left_inner_knuckle_link"/>
-			<axis xyz="0 0 1"/>
-			<origin xyz="0.06142 0.0127 0" rpy="${pi} 0.0 0.0" />
+		<joint name="${prefix}robotiq_85_left_inner_knuckle_joint" type="continuous">
+			<parent link="${prefix}robotiq_85_base_link"/>
+			<child link="${prefix}robotiq_85_left_inner_knuckle_link"/>
+			<axis xyz="0 0 1"/>
+			<origin xyz="0.06142 0.0127 0" rpy="${PI} 0.0 0.0" />
 			<limit lower="-3.14" upper="3.14" velocity="100.0" effort="0.1"/>
-			<mimic joint="robotiq_85_left_knuckle_joint" offset="0"/>
-		</joint>
-		<joint name="robotiq_85_right_inner_knuckle_joint" type="continuous">
-			<parent link="robotiq_85_base_link"/>
-			<child link="robotiq_85_right_inner_knuckle_link"/>
+			<mimic joint="${prefix}robotiq_85_left_knuckle_joint" offset="0"/>
+		</joint>
+		<xacro:mimic_joint_plugin_gazebo name_prefix="${prefix}robotiq_85_left_inner_knuckle_joint"
+			parent_joint="${prefix}robotiq_85_left_knuckle_joint" mimic_joint="${prefix}robotiq_85_left_inner_knuckle_joint"
+			multiplier="1.0" max_effort="10.0" />
+		<joint name="${prefix}robotiq_85_right_inner_knuckle_joint" type="continuous">
+			<parent link="${prefix}robotiq_85_base_link"/>
+			<child link="${prefix}robotiq_85_right_inner_knuckle_link"/>
 			<axis xyz="0 0 1"/>
 			<origin xyz="0.06142 -0.0127 0" rpy="0 0 0"/>
 			<limit lower="-3.14" upper="3.14" velocity="100.0" effort="0.1"/>
-			<mimic joint="robotiq_85_left_knuckle_joint" offset="0"/>
-		</joint>
-		<link name="robotiq_85_left_inner_knuckle_link">
+			<mimic joint="${prefix}robotiq_85_left_knuckle_joint" offset="0"/>
+		</joint>
+		<xacro:mimic_joint_plugin_gazebo name_prefix="${prefix}robotiq_85_right_inner_knuckle_joint"
+			parent_joint="${prefix}robotiq_85_left_knuckle_joint" mimic_joint="${prefix}robotiq_85_right_inner_knuckle_joint"
+			multiplier="1.0" max_effort="10.0" />
+		<link name="${prefix}robotiq_85_left_inner_knuckle_link">
 			<visual>
 				<geometry>
@@ -194,5 +233,5 @@
 			</inertial>
 		</link>
-		<link name="robotiq_85_right_inner_knuckle_link">
+		<link name="${prefix}robotiq_85_right_inner_knuckle_link">
 			<visual>
 				<geometry>
@@ -213,21 +252,27 @@
 			</inertial>
 		</link>
-		<joint name="robotiq_85_left_finger_tip_joint" type="continuous">
-			<parent link="robotiq_85_left_inner_knuckle_link"/>
-			<child link="robotiq_85_left_finger_tip_link"/>
+		<joint name="${prefix}robotiq_85_left_finger_tip_joint" type="continuous">
+			<parent link="${prefix}robotiq_85_left_inner_knuckle_link"/>
+			<child link="${prefix}robotiq_85_left_finger_tip_link"/>
 			<axis xyz="0 0 1"/>
 			<origin xyz="0.04303959807 -0.03759940821 0.0" rpy="0.0 0.0 0.0"/>
 			<limit lower="-3.14" upper="3.14" velocity="100.0" effort="0.1"/>
-			<mimic joint="robotiq_85_left_knuckle_joint" multiplier="-1"/>
-		</joint>
-		<joint name="robotiq_85_right_finger_tip_joint" type="continuous">
-			<parent link="robotiq_85_right_inner_knuckle_link"/>
-			<child link="robotiq_85_right_finger_tip_link"/>
+			<mimic joint="${prefix}robotiq_85_left_knuckle_joint" multiplier="-1"/>
+		</joint>
+		<xacro:mimic_joint_plugin_gazebo name_prefix="${prefix}robotiq_85_left_finger_tip_joint"
+			parent_joint="${prefix}robotiq_85_left_knuckle_joint" mimic_joint="${prefix}robotiq_85_left_finger_tip_joint"
+			multiplier="1.0" max_effort="10.0" />
+		<joint name="${prefix}robotiq_85_right_finger_tip_joint" type="continuous">
+			<parent link="${prefix}robotiq_85_right_inner_knuckle_link"/>
+			<child link="${prefix}robotiq_85_right_finger_tip_link"/>
 			<axis xyz="0 0 1"/>
 			<origin rpy="0.0 0.0 0.0" xyz="0.04303959807 -0.03759940821  0.0"/>
 			<limit lower="-3.14" upper="3.14" velocity="100.0" effort="0.1"/>
-			<mimic joint="robotiq_85_left_knuckle_joint" multiplier="-1"/>
-		</joint>
-		<link name="robotiq_85_left_finger_tip_link">
+			<mimic joint="${prefix}robotiq_85_left_knuckle_joint" multiplier="-1"/>
+		</joint>
+		<xacro:mimic_joint_plugin_gazebo name_prefix="${prefix}robotiq_85_right_finger_tip_joint"
+			parent_joint="${prefix}robotiq_85_left_knuckle_joint" mimic_joint="${prefix}robotiq_85_right_finger_tip_joint"
+			multiplier="1.0" max_effort="10.0" />
+		<link name="${prefix}robotiq_85_left_finger_tip_link">
 			<visual>
 				<geometry>
@@ -248,5 +293,5 @@
 			</inertial>
 		</link>
-		<gazebo reference="robotiq_85_left_finger_tip_link">
+		<gazebo reference="${prefix}robotiq_85_left_finger_tip_link">
 			<kp>1000000.0</kp>
 			<kd>100.0</kd>
@@ -257,5 +302,5 @@
 			<material>Gazebo/Grey</material>
 		</gazebo>
-		<link name="robotiq_85_right_finger_tip_link">
+		<link name="${prefix}robotiq_85_right_finger_tip_link">
 			<visual>
 				<geometry>
@@ -276,5 +321,5 @@
 			</inertial>
 		</link>
-		<gazebo reference="robotiq_85_right_finger_tip_link">
+		<gazebo reference="${prefix}robotiq_85_right_finger_tip_link">
 			<kp>1000000.0</kp>
 			<kd>100.0</kd>
@@ -285,5 +330,6 @@
 			<material>Gazebo/Grey</material>
 		</gazebo>
-		<xacro:robotiq_85_gripper_transmission />
+		<xacro:robotiq_85_gripper_transmission prefix="${prefix}" />
+	<!-- <xacro:robotiq_85_gripper_transmission /> -->
 		<joint name="robotiq_85_left_finger_tip_joint_mimic" type="fixed">
 			<parent link="world" />
@@ -311,4 +357,6 @@
 		</joint>
 		<link name="random5"/>
+		<!-- <xacro:robotiq_85_gripper_transmission_effort prefix="${prefix}" /> -->
+	</xacro:macro>
 	<!-- </xacro:macro> -->
 </robot>
