Commit message: eye-in-hand calibration added

File: src/yaskawa_mh5_description/urdf/TesseraVue_3D_sensor_bigger.urdf.xacro (robot description, xacro)
@@ -67,5 +67,6 @@
   <gazebo reference="tesseravue_camera_link">
     <sensor type="camera" name="TesseraVue">
-      <pose>0 0 0 0 0 0 </pose>
+      <!-- <pose>0 0 0 0 0 0 </pose> -->
+      <pose>0 0 0 0 1.57079632679 -1.57079632679</pose>
       <visualize>true</visualize>
       <update_rate>5.0</update_rate>

File: src/yaskawa_mh5_description/urdf/mh5.urdf.xacro (robot description, xacro)
@@ -7,4 +7,5 @@
   <xacro:include filename="$(find yaskawa_mh5_description)/urdf/robotiq_85_gripper.urdf.xacro"/>
   <!-- <xacro:include filename="$(find point_cloud_processing)/urdf/dynamic_object.urdf.xacro"/> -->
+  <!-- <xacro:include filename="$(find yaskawa_mh5_description)/urdf/cube_object.urdf.xacro"/> -->
 <!-- macro function for inertial-->
 	<xacro:macro name="default_inertial" params="mass">

File: src/yaskawa_mh5_description/urdf/mh5_gazebo.xacro (robot description, xacro)
@@ -5,4 +5,5 @@
         <plugin filename="libgazebo_ros2_control.so" name="gazebo_ros2_control">
             <robot_param>robot_description</robot_param>
+            <robot_param>object_description</robot_param>
             <robot_param_node>robot_state_publisher</robot_param_node>
             <parameters>$(find yaskawa_mh5_controller)/config/mh5_ros2_controller.yaml</parameters>

File: src/yaskawa_mh5_description/urdf/robotiq_85_gripper.ros2_control.xacro (robot description, xacro)
@@ -5,4 +5,5 @@
         <hardware>
             <plugin>gazebo_ros2_control/GazeboSystem</plugin>
+            <plugin name="gazebo_link_attacher" filename="libgazebo_link_attacher.so"/>
         </hardware>
             <joint name="robotiq_85_left_knuckle_joint">

File: src/yaskawa_mh5_description/urdf/robotiq_85_gripper.urdf.xacro (robot description, xacro)
@@ -7,31 +7,4 @@
         </plugin>
     </gazebo>
-<!--
-     <joint name="gripper_fixed" type="fixed">
-        <origin xyz="0 0 0" rpy="0 0 0"/>
-        <parent link="link_t"/>
-        <child link="gripper_root_link"/>
-    </joint> -->
-    <!-- <link name="gripper_root_link"> -->
-        <!-- <visual>
-            <origin xyz="0 0 0.5" rpy="0 0 0"/>
-            <geometry>
-                <box size="0.1 0.1 1.0"/>
-            </geometry>
-        </visual>
-        <collision>
-            <origin xyz="0 0 0.5" rpy="0 0 0"/>
-            <geometry>
-                <box size="0.1 0.1 1.0"/>
-            </geometry>
-        </collision>
-        <inertial>
-            <mass value="1e2" />
-            <origin xyz="0.0 0.0 0.0" />
-            <inertia ixx = "0.000001" ixy = "0.000000" ixz = "0.000000"
-                     iyx = "0.000000" iyy = "0.000001" iyz = "0.000000"
-                     izx = "0.000000" izy = "0.000000" izz = "0.000001" />
-        </inertial> -->
-    <!-- </link> -->
     <xacro:robotiq_85_gripper prefix="" parent="link_t" >
         <origin xyz="0.0 0.0 0.0" rpy="0 0 0"/>

File: src/yaskawa_mh5_description/urdf/robotiq_85_gripper_macro.urdf.xacro (robot description, xacro)
@@ -73,5 +73,5 @@
 			<axis xyz="0 0 1"/>
 			<origin rpy="${PI} 0.0 0.0" xyz="0.05490451627 0.03060114443 0.0"/>
-			<limit lower="0.0" upper="0.804" velocity="0.5" effort="50"/>
+			<limit lower="0.0" upper="0.804" velocity="5.0" effort="50"/>
 			<dynamics damping="100.0" />
 		</joint>
@@ -118,9 +118,10 @@
 			</collision>
 			<inertial>
-				<mass value="0.018491" />
-				<origin xyz="0.0 0.0 0.0" />
-				<inertia ixx = "0.000009" ixy = "-0.000001" ixz = "0.000000"
-					iyx = "-0.000001" iyy = "0.000001" iyz = "0.000000"
-					izx = "0.000000" izy = "0.000000" izz = "0.000010" />
+				<mass value="0.05" />
+				<origin xyz="0.0 0.0 0.0" />
+				 <inertia
+					ixx="2.0833e-06" ixy="0.0" ixz="0.0"
+					iyy="4.1667e-06" iyz="0.0"
+					izz="5.4167e-06"/>
 			</inertial>
 		</link>
@@ -137,9 +138,10 @@
 			</collision>
 			<inertial>
-				<mass value="0.018491" />
-				<origin xyz="0.0 0.0 0.0" />
-				<inertia ixx = "0.000009" ixy = "-0.000001" ixz = "0.000000"
-					iyx = "-0.000001" iyy = "0.000001" iyz = "0.000000"
-					izx = "0.000000" izy = "0.000000" izz = "0.000010" />
+				<mass value="0.05" />
+				<origin xyz="0.0 0.0 0.0" />
+				<inertia
+					ixx="2.0833e-06" ixy="0.0" ixz="0.0"
+					iyy="4.1667e-06" iyz="0.0"
+					izz="5.4167e-06"/>
 			</inertial>
 		</link>
